Commit message: fix: correct robot model names and remove version suffix
- Fix robot name in left hand models (was incorrectly set to "wujihand-right")
- Remove version suffix from robot name in all model files
- Update CHANGELOG.md for v0.3.0

File: urdf/right.urdf (robot description, URDF)
Before this commit: robot wujihand-right-v1.0.2, 26 links, 25 joints
Links:
- link right_finger1_link1: geometry collision mesh filename=right_finger1_link1.STL; visual mesh filename=right_finger1_link1.STL
- link right_finger1_link2: geometry collision mesh filename=right_finger1_link2.STL; visual mesh filename=right_finger1_link2.STL
- link right_finger1_link3: geometry collision mesh filename=right_finger1_link3.STL; visual mesh filename=right_finger1_link3.STL
- link right_finger1_link4: geometry collision mesh filename=right_finger1_link4.STL; visual mesh filename=right_finger1_link4.STL
- link right_finger1_tip_link: geometry collision mesh filename=right_finger1_tip_link.STL; visual mesh filename=right_finger1_tip_link.STL
- link right_finger2_link1: geometry collision mesh filename=right_finger2_link1.STL; visual mesh filename=right_finger2_link1.STL
- link right_finger2_link2: geometry collision mesh filename=right_finger2_link2.STL; visual mesh filename=right_finger2_link2.STL
- link right_finger2_link3: geometry collision mesh filename=right_finger2_link3.STL; visual mesh filename=right_finger2_link3.STL
- link right_finger2_link4: geometry collision mesh filename=right_finger2_link4.STL; visual mesh filename=right_finger2_link4.STL
- link right_finger2_tip_link: geometry collision mesh filename=right_finger2_tip_link.STL; visual mesh filename=right_finger2_tip_link.STL
- link right_finger3_link1: geometry collision mesh filename=right_finger3_link1.STL; visual mesh filename=right_finger3_link1.STL
- link right_finger3_link2: geometry collision mesh filename=right_finger3_link2.STL; visual mesh filename=right_finger3_link2.STL
- link right_finger3_link3: geometry collision mesh filename=right_finger3_link3.STL; visual mesh filename=right_finger3_link3.STL
- link right_finger3_link4: geometry collision mesh filename=right_finger3_link4.STL; visual mesh filename=right_finger3_link4.STL
- link right_finger3_tip_link: geometry collision mesh filename=right_finger3_tip_link.STL; visual mesh filename=right_finger3_tip_link.STL
- link right_finger4_link1: geometry collision mesh filename=right_finger4_link1.STL; visual mesh filename=right_finger4_link1.STL
- link right_finger4_link2: geometry collision mesh filename=right_finger4_link2.STL; visual mesh filename=right_finger4_link2.STL
- link right_finger4_link3: geometry collision mesh filename=right_finger4_link3.STL; visual mesh filename=right_finger4_link3.STL
- link right_finger4_link4: geometry collision mesh filename=right_finger4_link4.STL; visual mesh filename=right_finger4_link4.STL
- link right_finger4_tip_link: geometry collision mesh filename=right_finger4_tip_link.STL; visual mesh filename=right_finger4_tip_link.STL
- link right_finger5_link1: geometry collision mesh filename=right_finger5_link1.STL; visual mesh filename=right_finger5_link1.STL
- link right_finger5_link2: geometry collision mesh filename=right_finger5_link2.STL; visual mesh filename=right_finger5_link2.STL
- link right_finger5_link3: geometry collision mesh filename=right_finger5_link3.STL; visual mesh filename=right_finger5_link3.STL
- link right_finger5_link4: geometry collision mesh filename=right_finger5_link4.STL; visual mesh filename=right_finger5_link4.STL
- link right_finger5_tip_link: geometry collision mesh filename=right_finger5_tip_link.STL; visual mesh filename=right_finger5_tip_link.STL
- link right_palm_link: geometry collision mesh filename=right_palm_link.STL; visual mesh filename=right_palm_link.STL
