Commit message: fix: update URDF files

File: urdf/left.urdf (robot description, URDF)
Before this commit: robot wujihand-left, 26 links, 25 joints
Links:
- link left_finger1_link1: geometry collision mesh filename=../meshes/left/left_finger1_link1.STL; visual mesh filename=../meshes/left/left_finger1_link1.STL
- link left_finger1_link2: geometry collision mesh filename=../meshes/left/left_finger1_link2.STL; visual mesh filename=../meshes/left/left_finger1_link2.STL
- link left_finger1_link3: geometry collision mesh filename=../meshes/left/left_finger1_link3.STL; visual mesh filename=../meshes/left/left_finger1_link3.STL
- link left_finger1_link4: geometry collision mesh filename=../meshes/left/left_finger1_link4.STL; visual mesh filename=../meshes/left/left_finger1_link4.STL
- link left_finger1_tip_link: geometry collision mesh filename=../meshes/left/left_finger1_tip_link.STL; visual mesh filename=../meshes/left/left_finger1_tip_link.STL
- link left_finger2_link1: geometry collision mesh filename=../meshes/left/left_finger2_link1.STL; visual mesh filename=../meshes/left/left_finger2_link1.STL
- link left_finger2_link2: geometry collision mesh filename=../meshes/left/left_finger2_link2.STL; visual mesh filename=../meshes/left/left_finger2_link2.STL
- link left_finger2_link3: geometry collision mesh filename=../meshes/left/left_finger2_link3.STL; visual mesh filename=../meshes/left/left_finger2_link3.STL
- link left_finger2_link4: geometry collision mesh filename=../meshes/left/left_finger2_link4.STL; visual mesh filename=../meshes/left/left_finger2_link4.STL
- link left_finger2_tip_link: geometry collision mesh filename=../meshes/left/left_finger2_tip_link.STL; visual mesh filename=../meshes/left/left_finger2_tip_link.STL
- link left_finger3_link1: geometry collision mesh filename=../meshes/left/left_finger3_link1.STL; visual mesh filename=../meshes/left/left_finger3_link1.STL
- link left_finger3_link2: geometry collision mesh filename=../meshes/left/left_finger3_link2.STL; visual mesh filename=../meshes/left/left_finger3_link2.STL
- link left_finger3_link3: geometry collision mesh filename=../meshes/left/left_finger3_link3.STL; visual mesh filename=../meshes/left/left_finger3_link3.STL
- link left_finger3_link4: geometry collision mesh filename=../meshes/left/left_finger3_link4.STL; visual mesh filename=../meshes/left/left_finger3_link4.STL
- link left_finger3_tip_link: geometry collision mesh filename=../meshes/left/left_finger3_tip_link.STL; visual mesh filename=../meshes/left/left_finger3_tip_link.STL
- link left_finger4_link1: geometry collision mesh filename=../meshes/left/left_finger4_link1.STL; visual mesh filename=../meshes/left/left_finger4_link1.STL
- link left_finger4_link2: geometry collision mesh filename=../meshes/left/left_finger4_link2.STL; visual mesh filename=../meshes/left/left_finger4_link2.STL
- link left_finger4_link3: geometry collision mesh filename=../meshes/left/left_finger4_link3.STL; visual mesh filename=../meshes/left/left_finger4_link3.STL
- link left_finger4_link4: geometry collision mesh filename=../meshes/left/left_finger4_link4.STL; visual mesh filename=../meshes/left/left_finger4_link4.STL
- link left_finger4_tip_link: geometry collision mesh filename=../meshes/left/left_finger4_tip_link.STL; visual mesh filename=../meshes/left/left_finger4_tip_link.STL
- link left_finger5_link1: geometry collision mesh filename=../meshes/left/left_finger5_link1.STL; visual mesh filename=../meshes/left/left_finger5_link1.STL
- link left_finger5_link2: geometry collision mesh filename=../meshes/left/left_finger5_link2.STL; visual mesh filename=../meshes/left/left_finger5_link2.STL
- link left_finger5_link3: geometry collision mesh filename=../meshes/left/left_finger5_link3.STL; visual mesh filename=../meshes/left/left_finger5_link3.STL
- link left_finger5_link4: geometry collision mesh filename=../meshes/left/left_finger5_link4.STL; visual mesh filename=../meshes/left/left_finger5_link4.STL
- link left_finger5_tip_link: geometry collision mesh filename=../meshes/left/left_finger5_tip_link.STL; visual mesh filename=../meshes/left/left_finger5_tip_link.STL
- link left_palm_link: geometry collision mesh filename=../meshes/left/left_palm_link.STL; visual mesh filename=../meshes/left/left_palm_link.STL

File: urdf/right.urdf (robot description, URDF)
Before this commit: robot wujihand-right, 26 links, 25 joints
Links:
- link right_finger1_link1: geometry collision mesh filename=../meshes/right/right_finger1_link1.STL; visual mesh filename=../meshes/right/right_finger1_link1.STL
- link right_finger1_link2: geometry collision mesh filename=../meshes/right/right_finger1_link2.STL; visual mesh filename=../meshes/right/right_finger1_link2.STL
- link right_finger1_link3: geometry collision mesh filename=../meshes/right/right_finger1_link3.STL; visual mesh filename=../meshes/right/right_finger1_link3.STL
- link right_finger1_link4: geometry collision mesh filename=../meshes/right/right_finger1_link4.STL; visual mesh filename=../meshes/right/right_finger1_link4.STL
- link right_finger1_tip_link: geometry collision mesh filename=../meshes/right/right_finger1_tip_link.STL; visual mesh filename=../meshes/right/right_finger1_tip_link.STL
- link right_finger2_link1: geometry collision mesh filename=../meshes/right/right_finger2_link1.STL; visual mesh filename=../meshes/right/right_finger2_link1.STL
- link right_finger2_link2: geometry collision mesh filename=../meshes/right/right_finger2_link2.STL; visual mesh filename=../meshes/right/right_finger2_link2.STL
- link right_finger2_link3: geometry collision mesh filename=../meshes/right/right_finger2_link3.STL; visual mesh filename=../meshes/right/right_finger2_link3.STL
- link right_finger2_link4: geometry collision mesh filename=../meshes/right/right_finger2_link4.STL; visual mesh filename=../meshes/right/right_finger2_link4.STL
- link right_finger2_tip_link: geometry collision mesh filename=../meshes/right/right_finger2_tip_link.STL; visual mesh filename=../meshes/right/right_finger2_tip_link.STL
- link right_finger3_link1: geometry collision mesh filename=../meshes/right/right_finger3_link1.STL; visual mesh filename=../meshes/right/right_finger3_link1.STL
- link right_finger3_link2: geometry collision mesh filename=../meshes/right/right_finger3_link2.STL; visual mesh filename=../meshes/right/right_finger3_link2.STL
- link right_finger3_link3: geometry collision mesh filename=../meshes/right/right_finger3_link3.STL; visual mesh filename=../meshes/right/right_finger3_link3.STL
- link right_finger3_link4: geometry collision mesh filename=../meshes/right/right_finger3_link4.STL; visual mesh filename=../meshes/right/right_finger3_link4.STL
- link right_finger3_tip_link: geometry collision mesh filename=../meshes/right/right_finger3_tip_link.STL; visual mesh filename=../meshes/right/right_finger3_tip_link.STL
- link right_finger4_link1: geometry collision mesh filename=../meshes/right/right_finger4_link1.STL; visual mesh filename=../meshes/right/right_finger4_link1.STL
- link right_finger4_link2: geometry collision mesh filename=../meshes/right/right_finger4_link2.STL; visual mesh filename=../meshes/right/right_finger4_link2.STL
- link right_finger4_link3: geometry collision mesh filename=../meshes/right/right_finger4_link3.STL; visual mesh filename=../meshes/right/right_finger4_link3.STL
- link right_finger4_link4: geometry collision mesh filename=../meshes/right/right_finger4_link4.STL; visual mesh filename=../meshes/right/right_finger4_link4.STL
- link right_finger4_tip_link: geometry collision mesh filename=../meshes/right/right_finger4_tip_link.STL; visual mesh filename=../meshes/right/right_finger4_tip_link.STL
- link right_finger5_link1: geometry collision mesh filename=../meshes/right/right_finger5_link1.STL; visual mesh filename=../meshes/right/right_finger5_link1.STL
- link right_finger5_link2: geometry collision mesh filename=../meshes/right/right_finger5_link2.STL; visual mesh filename=../meshes/right/right_finger5_link2.STL
- link right_finger5_link3: geometry collision mesh filename=../meshes/right/right_finger5_link3.STL; visual mesh filename=../meshes/right/right_finger5_link3.STL
- link right_finger5_link4: geometry collision mesh filename=../meshes/right/right_finger5_link4.STL; visual mesh filename=../meshes/right/right_finger5_link4.STL
- link right_finger5_tip_link: geometry collision mesh filename=../meshes/right/right_finger5_tip_link.STL; visual mesh filename=../meshes/right/right_finger5_tip_link.STL
- link right_palm_link: geometry collision mesh filename=../meshes/right/right_palm_link.STL; visual mesh filename=../meshes/right/right_palm_link.STL

Commit message: fix: unify left/right hand joint limits using averaged values
Left and right hand URDF files had different joint limit values
(lower/upper) for all 20 joints, likely from independent calibration.

This commit unifies them by averaging the left and right values for
each joint, ensuring both hands have identical limit configurations.

File: urdf/left.urdf (robot description, URDF)
Before this commit: robot wujihand-left, 26 links, 25 joints
Joints:
- joint left_finger1_joint1: limit lower=0.0583 upper=1.5941 effort=0.4452 velocity=8.587 -> lower=0.0475 upper=1.6033 effort=0.4452 velocity=8.587
- joint left_finger1_joint2: limit lower=-0.1199 upper=0.9335 effort=0.4259 velocity=11.1 -> lower=-0.1387 upper=0.9324 effort=0.4259 velocity=11.1
- joint left_finger1_joint3: limit lower=-0.4646 upper=1.5639 effort=0.1888 velocity=13.578 -> lower=-0.4642 upper=1.5623 effort=0.1888 velocity=13.578
- joint left_finger1_joint4: limit lower=-0.4570 upper=1.5684 effort=0.1468 velocity=12.863 -> lower=-0.4699 upper=1.5568 effort=0.1468 velocity=12.863
- joint left_finger2_joint1: limit lower=-0.1560 upper=1.5619 effort=0.6188 velocity=8.203 -> lower=-0.1585 upper=1.5604 effort=0.6188 velocity=8.203
- joint left_finger2_joint2: limit lower=-0.4095 upper=0.2921 effort=0.1822 velocity=8.115 -> lower=-0.4069 upper=0.2988 effort=0.1822 velocity=8.115
- joint left_finger2_joint3: limit lower=-0.4839 upper=1.5466 effort=0.2251 velocity=13.578 -> lower=-0.4777 upper=1.5485 effort=0.2251 velocity=13.578
- joint left_finger2_joint4: limit lower=-0.4723 upper=1.5754 effort=0.2170 velocity=12.863 -> lower=-0.4683 upper=1.5753 effort=0.2170 velocity=12.863
- joint left_finger3_joint1: limit lower=-0.1569 upper=1.5536 effort=0.6494 velocity=8.203 -> lower=-0.1644 upper=1.5516 effort=0.6494 velocity=8.203
- joint left_finger3_joint2: limit lower=-0.3977 upper=0.3115 effort=0.1827 velocity=8.115 -> lower=-0.3995 upper=0.3055 effort=0.1827 velocity=8.115
- joint left_finger3_joint3: limit lower=-0.4847 upper=1.5411 effort=0.2078 velocity=13.578 -> lower=-0.4739 upper=1.5512 effort=0.2078 velocity=13.578
- joint left_finger3_joint4: limit lower=-0.4671 upper=1.5788 effort=0.2018 velocity=12.863 -> lower=-0.4684 upper=1.5745 effort=0.2018 velocity=12.863
- joint left_finger4_joint1: limit lower=-0.1507 upper=1.5636 effort=0.6389 velocity=8.203 -> lower=-0.1554 upper=1.5585 effort=0.6389 velocity=8.203
- joint left_finger4_joint2: limit lower=-0.4101 upper=0.3014 effort=0.1832 velocity=8.115 -> lower=-0.4118 upper=0.3087 effort=0.1832 velocity=8.115
- joint left_finger4_joint3: limit lower=-0.4747 upper=1.5526 effort=0.2249 velocity=13.578 -> lower=-0.4765 upper=1.5487 effort=0.2249 velocity=13.578
- joint left_finger4_joint4: limit lower=-0.4729 upper=1.5718 effort=0.2044 velocity=12.863 -> lower=-0.4777 upper=1.5634 effort=0.2044 velocity=12.863
- joint left_finger5_joint1: limit lower=-0.1578 upper=1.5632 effort=0.6441 velocity=8.203 -> lower=-0.1626 upper=1.5585 effort=0.6441 velocity=8.203
- joint left_finger5_joint2: limit lower=-0.4103 upper=0.2949 effort=0.1798 velocity=8.115 -> lower=-0.4153 upper=0.2940 effort=0.1798 velocity=8.115
- joint left_finger5_joint3: limit lower=-0.4733 upper=1.5560 effort=0.2384 velocity=13.578 -> lower=-0.4768 upper=1.5490 effort=0.2384 velocity=13.578
- joint left_finger5_joint4: limit lower=-0.4662 upper=1.5760 effort=0.1866 velocity=12.863 -> lower=-0.4683 upper=1.5735 effort=0.1866 velocity=12.863

File: urdf/right.urdf (robot description, URDF)
Before this commit: robot wujihand-right, 26 links, 25 joints
Joints:
- joint right_finger1_joint1: limit lower=0.0368 upper=1.6125 effort=0.4452 velocity=8.58701992 -> lower=0.0475 upper=1.6033 effort=0.4452 velocity=8.58701992
- joint right_finger1_joint2: limit lower=-0.1576 upper=0.9312 effort=0.4259 velocity=11.10029404 -> lower=-0.1387 upper=0.9324 effort=0.4259 velocity=11.10029404
- joint right_finger1_joint3: limit lower=-0.4638 upper=1.5607 effort=0.1888 velocity=12.86307659 -> lower=-0.4642 upper=1.5623 effort=0.1888 velocity=12.86307659
- joint right_finger1_joint4: limit lower=-0.4829 upper=1.5451 effort=0.1468 velocity=13.57866158 -> lower=-0.4699 upper=1.5568 effort=0.1468 velocity=13.57866158
- joint right_finger2_joint1: limit lower=-0.1611 upper=1.5588 effort=0.6188 velocity=8.203047484 -> lower=-0.1585 upper=1.5604 effort=0.6188 velocity=8.203047484
- joint right_finger2_joint2: limit lower=-0.4044 upper=0.3054 effort=0.1822 velocity=8.115781022 -> lower=-0.4069 upper=0.2988 effort=0.1822 velocity=8.115781022
- joint right_finger2_joint3: limit lower=-0.4714 upper=1.5504 effort=0.2251 velocity=12.86307659 -> lower=-0.4777 upper=1.5485 effort=0.2251 velocity=12.86307659
- joint right_finger2_joint4: limit lower=-0.4644 upper=1.5753 effort=0.2170 velocity=13.57866158 -> lower=-0.4683 upper=1.5753 effort=0.2170 velocity=13.57866158
- joint right_finger3_joint1: limit lower=-0.1719 upper=1.5496 effort=0.6494 velocity=8.203047484 -> lower=-0.1644 upper=1.5516 effort=0.6494 velocity=8.203047484
- joint right_finger3_joint2: limit lower=-0.4014 upper=0.2996 effort=0.1827 velocity=8.115781022 -> lower=-0.3995 upper=0.3055 effort=0.1827 velocity=8.115781022
- joint right_finger3_joint3: limit lower=-0.4632 upper=1.5613 effort=0.2078 velocity=12.86307659 -> lower=-0.4739 upper=1.5512 effort=0.2078 velocity=12.86307659
- joint right_finger3_joint4: limit lower=-0.4697 upper=1.5702 effort=0.2018 velocity=13.57866158 -> lower=-0.4684 upper=1.5745 effort=0.2018 velocity=13.57866158
- joint right_finger4_joint1: limit lower=-0.1601 upper=1.5534 effort=0.6389 velocity=8.203047484 -> lower=-0.1554 upper=1.5585 effort=0.6389 velocity=8.203047484
- joint right_finger4_joint2: limit lower=-0.4134 upper=0.3161 effort=0.1832 velocity=8.115781022 -> lower=-0.4118 upper=0.3087 effort=0.1832 velocity=8.115781022
- joint right_finger4_joint3: limit lower=-0.4782 upper=1.5448 effort=0.2249 velocity=12.86307659 -> lower=-0.4765 upper=1.5487 effort=0.2249 velocity=12.86307659
- joint right_finger4_joint4: limit lower=-0.4825 upper=1.5550 effort=0.2044 velocity=13.57866158 -> lower=-0.4777 upper=1.5634 effort=0.2044 velocity=13.57866158
- joint right_finger5_joint1: limit lower=-0.1674 upper=1.5539 effort=0.6441 velocity=8.203047484 -> lower=-0.1626 upper=1.5585 effort=0.6441 velocity=8.203047484
- joint right_finger5_joint2: limit lower=-0.4203 upper=0.2931 effort=0.1798 velocity=8.115781022 -> lower=-0.4153 upper=0.2940 effort=0.1798 velocity=8.115781022
- joint right_finger5_joint3: limit lower=-0.4804 upper=1.5420 effort=0.2384 velocity=12.86307659 -> lower=-0.4768 upper=1.5490 effort=0.2384 velocity=12.86307659
- joint right_finger5_joint4: limit lower=-0.4705 upper=1.5709 effort=0.1866 velocity=13.57866158 -> lower=-0.4683 upper=1.5735 effort=0.1866 velocity=13.57866158
