Commit message: Adjust right index MCP2 limits

File: urdf/right-ros.urdf (robot description, URDF)
Before this commit: robot wujihand-right, 26 links, 25 joints
Joints:
- joint right_finger2_joint2: limit lower=-0.4044 upper=0.3054 effort=0.1822 velocity=8.115781022 -> lower=-0.292 upper=0.409 effort=0.1822 velocity=8.115781022

File: urdf/right.urdf (robot description, URDF)
Before this commit: robot wujihand-right, 26 links, 25 joints
Joints:
- joint right_finger2_joint2: limit lower=-0.4044 upper=0.3054 effort=0.1822 velocity=8.115781022 -> lower=-0.292 upper=0.409 effort=0.1822 velocity=8.115781022
