Commit message: feat: replace hand description with WH120 model
- Replace right hand meshes and URDFs with WH120 version
- Remove left hand files (meshes, mjcf, launch, urdf)
- Remove collision meshes (visual only)
- Update right.xml MJCF with WH120 kinematics
- Fix finger5_joint1 and finger5_joint4 axis direction

Co-Authored-By: Claude Opus 4.5 <noreply@anthropic.com>

File: urdf/right-ros.urdf (robot description, URDF)
Before this commit: robot wujihand-right-v1.0.2, 26 links, 25 joints
Links:
- removed link finger1_link1
- removed link finger1_link2
- removed link finger1_link3
- removed link finger1_link4
- removed link finger1_tip_link
- removed link finger2_link1
- removed link finger2_link2
- removed link finger2_link3
- removed link finger2_link4
- removed link finger2_tip_link
- removed link finger3_link1
- removed link finger3_link2
- removed link finger3_link3
- removed link finger3_link4
- removed link finger3_tip_link
- removed link finger4_link1
- removed link finger4_link2
- removed link finger4_link3
- removed link finger4_link4
- removed link finger4_tip_link
- removed link finger5_link1
- removed link finger5_link2
- removed link finger5_link3
- removed link finger5_link4
- removed link finger5_tip_link
- removed link palm_link
- added link right_finger1_link1, mass 0.0075; collision mesh filename=package://wuji_hand_description/meshes/right/right_finger1_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; visual mesh filename=package://wuji_hand_description/meshes/right/right_finger1_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
- added link right_finger1_link2, mass 0.0248; collision mesh filename=package://wuji_hand_description/meshes/right/right_finger1_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; visual mesh filename=package://wuji_hand_description/meshes/right/right_finger1_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
- added link right_finger1_link3, mass 0.0165; collision mesh filename=package://wuji_hand_description/meshes/right/right_finger1_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; visual mesh filename=package://wuji_hand_description/meshes/right/right_finger1_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
- added link right_finger1_link4, mass 0.0165; collision mesh filename=package://wuji_hand_description/meshes/right/right_finger1_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; visual mesh filename=package://wuji_hand_description/meshes/right/right_finger1_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
- added link right_finger1_tip_link, mass 0.0041; collision mesh filename=package://wuji_hand_description/meshes/right/right_finger1_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; visual mesh filename=package://wuji_hand_description/meshes/right/right_finger1_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
- added link right_finger2_link1, mass 0.0032; collision mesh filename=package://wuji_hand_description/meshes/right/right_finger2_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; visual mesh filename=package://wuji_hand_description/meshes/right/right_finger2_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
- added link right_finger2_link2, mass 0.033; collision mesh filename=package://wuji_hand_description/meshes/right/right_finger2_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; visual mesh filename=package://wuji_hand_description/meshes/right/right_finger2_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
- added link right_finger2_link3, mass 0.0165; collision mesh filename=package://wuji_hand_description/meshes/right/right_finger2_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; visual mesh filename=package://wuji_hand_description/meshes/right/right_finger2_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
- added link right_finger2_link4, mass 0.014; collision mesh filename=package://wuji_hand_description/meshes/right/right_finger2_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; visual mesh filename=package://wuji_hand_description/meshes/right/right_finger2_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
- added link right_finger2_tip_link, mass 0.00318; collision mesh filename=package://wuji_hand_description/meshes/right/right_finger2_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; visual mesh filename=package://wuji_hand_description/meshes/right/right_finger2_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
- added link right_finger3_link1, mass 0.0032; collision mesh filename=package://wuji_hand_description/meshes/right/right_finger3_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; visual mesh filename=package://wuji_hand_description/meshes/right/right_finger3_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
- added link right_finger3_link2, mass 0.033; collision mesh filename=package://wuji_hand_description/meshes/right/right_finger3_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; visual mesh filename=package://wuji_hand_description/meshes/right/right_finger3_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
- added link right_finger3_link3, mass 0.0165; collision mesh filename=package://wuji_hand_description/meshes/right/right_finger3_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; visual mesh filename=package://wuji_hand_description/meshes/right/right_finger3_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
- added link right_finger3_link4, mass 0.014; collision mesh filename=package://wuji_hand_description/meshes/right/right_finger3_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; visual mesh filename=package://wuji_hand_description/meshes/right/right_finger3_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
- added link right_finger3_tip_link, mass 0.00318; collision mesh filename=package://wuji_hand_description/meshes/right/right_finger3_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; visual mesh filename=package://wuji_hand_description/meshes/right/right_finger3_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
- added link right_finger4_link1, mass 0.0032; collision mesh filename=package://wuji_hand_description/meshes/right/right_finger4_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; visual mesh filename=package://wuji_hand_description/meshes/right/right_finger4_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
- added link right_finger4_link2, mass 0.033; collision mesh filename=package://wuji_hand_description/meshes/right/right_finger4_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; visual mesh filename=package://wuji_hand_description/meshes/right/right_finger4_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
- added link right_finger4_link3, mass 0.0165; collision mesh filename=package://wuji_hand_description/meshes/right/right_finger4_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; visual mesh filename=package://wuji_hand_description/meshes/right/right_finger4_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
- added link right_finger4_link4, mass 0.014; collision mesh filename=package://wuji_hand_description/meshes/right/right_finger4_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; visual mesh filename=package://wuji_hand_description/meshes/right/right_finger4_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
- added link right_finger4_tip_link, mass 0.00318; collision mesh filename=package://wuji_hand_description/meshes/right/right_finger4_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; visual mesh filename=package://wuji_hand_description/meshes/right/right_finger4_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
- added link right_finger5_link1, mass 0.0032; collision mesh filename=package://wuji_hand_description/meshes/right/right_finger5_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; visual mesh filename=package://wuji_hand_description/meshes/right/right_finger5_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
- added link right_finger5_link2, mass 0.033; collision mesh filename=package://wuji_hand_description/meshes/right/right_finger5_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; visual mesh filename=package://wuji_hand_description/meshes/right/right_finger5_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
- added link right_finger5_link3, mass 0.0165; collision mesh filename=package://wuji_hand_description/meshes/right/right_finger5_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; visual mesh filename=package://wuji_hand_description/meshes/right/right_finger5_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
- added link right_finger5_link4, mass 0.014; collision mesh filename=package://wuji_hand_description/meshes/right/right_finger5_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; visual mesh filename=package://wuji_hand_description/meshes/right/right_finger5_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
- added link right_finger5_tip_link, mass 0.00318; collision mesh filename=package://wuji_hand_description/meshes/right/right_finger5_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; visual mesh filename=package://wuji_hand_description/meshes/right/right_finger5_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
- added link right_palm_link, mass 0.16914; collision mesh filename=package://wuji_hand_description/meshes/right/right_palm_lin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; visual mesh filename=package://wuji_hand_description/meshes/right/right_palm_lin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
Joints:
- removed joint finger1_joint1
- removed joint finger1_joint2
- removed joint finger1_joint3
- removed joint finger1_joint4
- removed joint finger1_tip_fixed
- removed joint finger2_joint1
- removed joint finger2_joint2
- removed joint finger2_joint3
- removed joint finger2_joint4
- removed joint finger2_tip_fixed
- removed joint finger3_joint1
- removed joint finger3_joint2
- removed joint finger3_joint3
- removed joint finger3_joint4
- removed joint finger3_tip_fixed
- removed joint finger4_joint1
- removed joint finger4_joint2
- removed joint finger4_joint3
- removed joint finger4_joint4
- removed joint finger4_tip_fixed
- removed joint finger5_joint1
- removed joint finger5_joint2
- removed joint finger5_joint3
- removed joint finger5_joint4
- removed joint finger5_tip_fixed
- added joint right_finger1_joint1: type revolute, parent right_palm_link, child right_finger1_link1, origin xyz=0.0081297 0.017208 0.016463 rpy=1.942 -1.0586 2.7208, axis -1 0 0, limit lower=0.0368 upper=1.6125 effort=0.4452 velocity=8.587
- added joint right_finger1_joint2: type revolute, parent right_finger1_link1, child right_finger1_link2, origin xyz=-0.00024788 0.003574 0.014324 rpy=0.744 0.43559 1.6887, axis 1 0 0, limit lower=-0.1576 upper=0.9312 effort=0.4259 velocity=11.1
- added joint right_finger1_joint3: type revolute, parent right_finger1_link2, child right_finger1_link3, origin xyz=0 0 0.0325 rpy=0.087266 0 -0.56723, axis 0 1 0, limit lower=-0.4638 upper=1.5607 effort=0.1888 velocity=12.86
- added joint right_finger1_joint4: type revolute, parent right_finger1_link3, child right_finger1_link4, origin xyz=0 -5E-05 0.035 rpy=0 0 0, axis 0 1 0, limit lower=-0.4829 upper=1.5451 effort=0.1468 velocity=13.5
- added joint right_finger1_tip_fixed: type fixed, parent right_finger1_link4, child right_finger1_tip_link, origin xyz=-0.00055745 0 0.027697 rpy=0 0 0, axis 0 0 0
- added joint right_finger2_joint1: type revolute, parent right_palm_link, child right_finger2_link1, origin xyz=-0.0033601 0.022653 0.069976 rpy=-0.137 -0.039905 -0.094973, axis 0 1 0, limit lower=-0.1611 upper=1.5588 effort=0.6188 velocity=8.203
- added joint right_finger2_joint2: type revolute, parent right_finger2_link1, child right_finger2_link2, origin xyz=-0.001201 0 0.0145 rpy=0 0 0, axis -1 0 0, limit lower=-0.4044 upper=0.3054 effort=0.1822 velocity=8.11
- added joint right_finger2_joint3: type revolute, parent right_finger2_link2, child right_finger2_link3, origin xyz=0 0 0.0376000000000015 rpy=0 0 0, axis 0 1 0, limit lower=-0.4714 upper=1.5504 effort=0.2251 velocity=12.86
- added joint right_finger2_joint4: type revolute, parent right_finger2_link3, child right_finger2_link4, origin xyz=0 0 0.0295 rpy=0 0 0, axis 0 1 0, limit lower=-0.4644 upper=1.5753 effort=0.2170 velocity=13.5
- added joint right_finger2_tip_fixed: type fixed, parent right_finger2_link4, child right_finger2_tip_link, origin xyz=-0.00167219746761749 0 0.0250000000000001 rpy=0 0 0, axis 0 0 0
- added joint right_finger3_joint1: type revolute, parent right_palm_link, child right_finger3_link1, origin xyz=-0.0083399 0.00094389 0.073911 rpy=0.011153 -0.034411 0.00033712, axis 0 1 0, limit lower=-0.1719 upper=1.5496 effort=0.6494 velocity=8.203
- added joint right_finger3_joint2: type revolute, parent right_finger3_link1, child right_finger3_link2, origin xyz=-0.00120098018725689 0 0.0145000000001074 rpy=0 0 0, axis -1 0 0, limit lower=-0.4014 upper=0.2996 effort=0.1827 velocity=8.11
- added joint right_finger3_joint3: type revolute, parent right_finger3_link2, child right_finger3_link3, origin xyz=0 0 0.0376 rpy=0 0 0, axis 0 1 0, limit lower=-0.4632 upper=1.5613 effort=0.2078 velocity=12.86
- added joint right_finger3_joint4: type revolute, parent right_finger3_link3, child right_finger3_link4, origin xyz=0 0 0.0295 rpy=0 0 0, axis 0 1 0, limit lower=-0.4697 upper=1.5702 effort=0.2018 velocity=13.5
- added joint right_finger3_tip_fixed: type fixed, parent right_finger3_link4, child right_finger3_tip_link, origin xyz=-0.0016722 0 0.025 rpy=0 0 1.5689, axis 0 0 0
- added joint right_finger4_joint1: type revolute, parent right_palm_link, child right_finger4_link1, origin xyz=-0.0056256 -0.019751 0.065395 rpy=0.14173 -0.016994 0.065967, axis 0 1 0, limit lower=-0.1601 upper=1.5534 effort=0.6389 velocity=8.203
- added joint right_finger4_joint2: type revolute, parent right_finger4_link1, child right_finger4_link2, origin xyz=-0.001201 0 0.0145 rpy=0 0 0, axis -1 0 0, limit lower=-0.4134 upper=0.3161 effort=0.1832 velocity=8.11
- added joint right_finger4_joint3: type revolute, parent right_finger4_link2, child right_finger4_link3, origin xyz=0 0 0.0376000000000015 rpy=0 0 0, axis 0 1 0, limit lower=-0.4782 upper=1.5448 effort=0.2249 velocity=12.86
- added joint right_finger4_joint4: type revolute, parent right_finger4_link3, child right_finger4_link4, origin xyz=0 0 0.0295 rpy=0 0 0, axis 0 1 0, limit lower=-0.4825 upper=1.5550 effort=0.2044 velocity=13.5
- added joint right_finger4_tip_fixed: type fixed, parent right_finger4_link4, child right_finger4_tip_link, origin xyz=-0.00167219746761747 0 0.025 rpy=0 0 -1.8672163655129, axis 0 0 0
- added joint right_finger5_joint1: type revolute, parent right_palm_link, child right_finger5_link1, origin xyz=-0.000761381007086758 -0.0373566917530012 0.0552917300142485 rpy=0.248910111063835 -0.0100079660367069 0.133606798058913, axis 0 1 0, limit lower=-0.1674 upper=1.5539 effort=0.6441 velocity=8.203
- added joint right_finger5_joint2: type revolute, parent right_finger5_link1, child right_finger5_link2, origin xyz=-0.00120098018724168 0 0.0145000000001571 rpy=0.0106031882018288 0 0, axis -1 0 0, limit lower=-0.4203 upper=0.2931 effort=0.1798 velocity=8.11
- added joint right_finger5_joint3: type revolute, parent right_finger5_link2, child right_finger5_link3, origin xyz=0 0.000456254826584512 0.0335970509350638 rpy=-0.0106031882018287 0 0, axis 0 1 0, limit lower=-0.4804 upper=1.5420 effort=0.2384 velocity=12.86
- added joint right_finger5_joint4: type revolute, parent right_finger5_link3, child right_finger5_link4, origin xyz=0 0 0.0275000000000001 rpy=0 0 0, axis 0 1 0, limit lower=-0.4705 upper=1.5709 effort=0.1866 velocity=13.5
- added joint right_finger5_tip_fixed: type fixed, parent right_finger5_link4, child right_finger5_tip_link, origin xyz=-0.00167219746761757 0 0.025 rpy=0 0 0, axis 0 0 0
