Commit message: Fix/left right hand urdf inconsistency (#33)
* feat: update URDF/MJCF/meshes with calibrated model from urdf_cali pipeline

Replace all model files with sysid-calibrated versions from urdf_cali/reference/result:
- MJCF: updated joint defaults (armature, damping), per-joint actuator params, axis corrections
- URDF (non-ROS + ROS): calibrated inertia, joint limits, axis fixes, preserved mujoco compiler block
- Meshes: synced STL files from calibration pipeline output

Co-Authored-By: Claude Opus 4.6 (1M context) <noreply@anthropic.com>

* chore: refresh configuration wujihand base/physics USD

Regenerate usd/{left,right}/configuration/wujihand_{base,physics}.usd
after the latest URDF update so the IsaacLab configuration layer
reflects the calibrated model.

Co-Authored-By: Claude Opus 4.6 (1M context) <noreply@anthropic.com>

* feat: add docking folder with meshes, mjcf, urdf, and usd assets

Co-Authored-By: Claude Sonnet 4.6 <noreply@anthropic.com>

* feat: update docs and build config for docking module

- Add docking/ to CMakeLists.txt install targets
- Add docking/ to README repository structure
- Add docking module entry to CHANGELOG [Unreleased]

Co-Authored-By: Claude Sonnet 4.6 <noreply@anthropic.com>

* fix: drop rogue limit blocks, correct docking-ros path, install mjcf/usd

Apply hotfixes to the model description on top of the sysid calibration
pass in 62b85a6:

- urdf/right.urdf, urdf/right-ros.urdf: remove spurious <limit> elements
  from the five *_finger*_tip_fixed joints. URDF <limit> is only defined
  for revolute/prismatic joints; these 25 lines were the entire structural
  asymmetry between the left and right hand URDFs, which defeats the
  stated purpose of this branch. Root cause lives in the upstream
  urdf_cali pipeline (update_joint_limits.py) and is filed separately.

- docking/urdf/docking-ros.urdf: fix wrong ROS package reference. Mesh
  paths now use package://wuji_hand_description/docking/meshes/... to
  match the installed share/ layout. Previous package://wuji_description/
  robots/docking/meshes/... would have failed to resolve after colcon
  build because the package name is wuji_hand_description and there is
  no robots/ prefix.

- CMakeLists.txt: also install mjcf/ and usd/ so MuJoCo and Isaac Sim
  assets ship with the ROS package.

- README.md: document how to preview the new docking module.

- CHANGELOG.md: add entries for all of the above under [Unreleased].

Co-Authored-By: Claude Opus 4.6 (1M context) <noreply@anthropic.com>

* fix(mjcf): clamp actuator ctrlrange to exact joint range

Seven ctrlrange upper bounds in mjcf/right.xml and eight in mjcf/left.xml
exceeded their corresponding joint's hard range by ~5e-4 rad because the
calibration exporter truncated ctrlrange to three decimals while the
joint range was emitted with four. A position controller saturated at
such a bound would keep chasing an unreachable target and cause jitter
near the joint stops.

Rewrite each offending ctrlrange so it matches the joint range string
exactly; leave everything else (kp, kv, forcerange, joint ordering)
untouched. Post-fix verification: every actuator's ctrlrange now lies
within its joint range, and both MJCF files still parse as valid XML.

Addresses CodeRabbit review 4089329830 (PR #33). Root cause lives in
the upstream urdf_cali pipeline and will be fixed there separately.

Co-Authored-By: Claude Opus 4.6 (1M context) <noreply@anthropic.com>

---------

Co-authored-by: AIRJASON50 <1543670713@qq.com>
Co-authored-by: Claude Opus 4.6 (1M context) <noreply@anthropic.com>
Co-authored-by: qqsq1232 <932851972@qq.com>

File: urdf/right-ros.urdf (robot description, URDF)
Before this commit: robot wujihand-right, 26 links, 25 joints
Joints:
- joint right_finger1_joint1: axis -0 1 -0 -> 0 1 0; limit lower=0.0368 upper=1.6125 effort=0.4452 velocity=8.58701992 -> lower=0.0368 upper=1.6125 effort=0.4452 velocity=8.587; origin xyz=0.0085244 0.020575 0.028712 rpy=-1.328 -0.37161 -0.7307 -> xyz=0.0084398536891496 0.0205866432770798 0.0288928344360424 rpy=-1.32802443797267 -0.371613529401197 -0.730700470955738
- joint right_finger1_joint2: axis -0 -1 -0 -> 0 1 0; limit lower=-0.1576 upper=0.9312 effort=0.4259 velocity=11.10029404 -> lower=-0.1576 upper=0.9312 effort=0.4259 velocity=11.1; origin xyz=-0.0047549 -0.0060191 0.014132 rpy=-0.57428 -0.23677 1.8034 -> xyz=-0.00475489769909336 -0.00581913700106552 0.0141320977693281 rpy=0.574275025049342 0.236773483165491 -1.3381949894783
- joint right_finger1_joint3: limit lower=-0.4638 upper=1.5607 effort=0.1888 velocity=12.86307659 -> lower=-0.4638 upper=1.5607 effort=0.1888 velocity=12.863; origin xyz=0.00018873 -0.0009916 0.034664 rpy=0.049049 0.017311 -1.9085 -> xyz=-0.000266709908258896 0.000991501558320149 0.0346656189847898 rpy=0.0490494507279648 0.017311243665607 1.23305222676766
- joint right_finger1_joint4: limit lower=-0.4829 upper=1.5451 effort=0.1468 velocity=13.57866158 -> lower=-0.4829 upper=1.5451 effort=0.1468 velocity=13.578; origin xyz=0 -0.00025 0.0295 rpy=0 0 0 -> xyz=0 0.000200000007014398 0.0295000000021542 rpy=0 0 0
- joint right_finger1_tip_fixed: origin xyz=-0.0011048 0.00023218 0.0283 rpy=0 0 0 -> xyz=-0.00105000000124529 -0.000200000000000502 0.0272999999978436 rpy=0 0 0
- joint right_finger2_joint1: limit lower=-0.1611 upper=1.5588 effort=0.6188 velocity=8.203047484 -> lower=-0.1611 upper=1.5588 effort=0.6188 velocity=8.203; origin xyz=-0.0058701 0.029434 0.091917 rpy=-0.11071 -0.071139 -0.21822 -> xyz=-0.00587008921485247 0.0294338632809287 0.0919165306699325 rpy=-0.110709283985856 -0.0711392458057915 -0.218224846691839
- joint right_finger2_joint2: axis -1 0 0 -> 0 0.999999999978991 0; limit lower=-0.37 upper=0.37 effort=0.1822 velocity=8.115781022 -> lower=-0.4044 upper=0.3054 effort=0.1822 velocity=8.1158; origin xyz=0.0022 0 0.004 rpy=0 0 0 -> xyz=0.00220000016749383 0 0.00400000572323159 rpy=0 0 1.57079633736728
- joint right_finger2_joint3: axis -0 1 -0 -> 0 1 0; limit lower=-0.4714 upper=1.5504 effort=0.2251 velocity=12.86307659 -> lower=-0.4714 upper=1.5504 effort=0.2251 velocity=12.863; origin xyz=-0.0047503 0 0.043618 rpy=0 0 -0.00026861 -> xyz=0 0.00475028218260664 0.0436176566595782 rpy=0 0 -1.57106495008262
- joint right_finger2_joint4: axis -0 1 -0 -> 0 1 0; limit lower=-0.4644 upper=1.5753 effort=0.2170 velocity=13.57866158 -> lower=-0.4644 upper=1.5753 effort=0.2170 velocity=13.578; origin xyz=0 0 0.0295 rpy=0 0 0 -> xyz=0 -0.00020000000636031 0.0294999999999844 rpy=0 0 0
- joint right_finger2_tip_fixed: origin xyz=-0.00105 0 0.0274 rpy=0 0 0 -> xyz=-0.00104999999940632 0.000200000000000138 0.0266999989308851 rpy=0 0 0
- joint right_finger3_joint1: limit lower=-0.1719 upper=1.5496 effort=0.6494 velocity=8.203047484 -> lower=-0.1719 upper=1.5496 effort=0.6494 velocity=8.203; origin xyz=-0.01046 0.0074615 0.089544 rpy=-5.0886E-05 -0.087266 0.00058387 -> xyz=-0.0104597238611628 0.00746146014385576 0.0895435117703666 rpy=-5.08864726421373E-05 -0.0872664633653732 0.000583871740007801
- joint right_finger3_joint2: axis -1 0 0 -> 0 1 0; limit lower=-0.37 upper=0.37 effort=0.1827 velocity=8.115781022 -> lower=-0.4014 upper=0.2996 effort=0.1827 velocity=8.1158; origin xyz=0.0022 0 0.004 rpy=0 0 0 -> xyz=0.00220000049491006 0 0.00400000560544524 rpy=0 0 1.57079633736875
- joint right_finger3_joint3: axis -0 1 -0 -> 0 1 0; limit lower=-0.4632 upper=1.5613 effort=0.2078 velocity=12.86307659 -> lower=-0.4632 upper=1.5613 effort=0.2078 velocity=12.863; origin xyz=-0.00475 0 0.043618 rpy=0 0 -0.00026861 -> xyz=0 0.0047500001855858 0.0436176873657041 rpy=0 0 -1.57106495008262
- joint right_finger3_joint4: axis -0 1 -0 -> 0 1 0; limit lower=-0.4697 upper=1.5702 effort=0.2018 velocity=13.57866158 -> lower=-0.4697 upper=1.5702 effort=0.2018 velocity=13.579; origin xyz=0 0 0.0295 rpy=0 0 0 -> xyz=0 -0.000200000004070615 0.0294999999999999 rpy=0 0 0
- joint right_finger3_tip_fixed: origin xyz=-0.0010491 0 0.0267 rpy=0 0 0 -> xyz=-0.00104908716153243 0.000201039517772421 0.0266999998992792 rpy=0 0 0
- joint right_finger4_joint1: axis -0 1 -0 -> 0 1 0; limit lower=-0.1601 upper=1.5534 effort=0.6389 velocity=8.203047484 -> lower=-0.1601 upper=1.5534 effort=0.6389 velocity=8.203; origin xyz=-0.0076649 -0.013712 0.084429 rpy=0.090375 -0.083436 0.047127 -> xyz=-0.0076648599285041 -0.0137122383759844 0.084428694586379 rpy=0.0903746211775801 -0.0834355030065636 0.0471266290291302
- joint right_finger4_joint2: axis -1 0 0 -> 0 1 0; limit lower=-0.37 upper=0.37 effort=0.1832 velocity=8.115781022 -> lower=-0.4134 upper=0.3161 effort=0.1832 velocity=8.1158; origin xyz=0.0022 0 0.004 rpy=0 0 0 -> xyz=0.00220000052979842 0 0.00400000547923511 rpy=0 0 1.57079633736852
- joint right_finger4_joint3: axis -0 1 -0 -> 0 1 0; limit lower=-0.4782 upper=1.5448 effort=0.2249 velocity=12.86307659 -> lower=-0.4782 upper=1.5448 effort=0.2249 velocity=12.863; origin xyz=-0.00475 0 0.043618 rpy=0 0 -0.00026861 -> xyz=0 0.00474999949683786 0.0436176874505065 rpy=0 0 -1.57106495008262
- joint right_finger4_joint4: axis -0 1 -0 -> 0 1 0; limit lower=-0.4825 upper=1.5550 effort=0.2044 velocity=13.57866158 -> lower=-0.4825 upper=1.5550 effort=0.2044 velocity=13.579; origin xyz=0 0 0.0295 rpy=0 0 0 -> xyz=0 -0.000200000003294468 0.0294999999999999 rpy=0 0 0
- joint right_finger4_tip_fixed: origin xyz=-0.0010528 0 0.0267 rpy=0 0 0 -> xyz=-0.00105960974768627 0.000190450796499008 0.0266999999370233 rpy=0 0 0
- joint right_finger5_joint1: limit lower=-0.1674 upper=1.5539 effort=0.6441 velocity=8.203047484 -> lower=-0.1674 upper=1.5539 effort=0.6441 velocity=8.203; origin xyz=-0.0022687 -0.034001 0.074281 rpy=0.19248 -0.092517 0.15767 -> xyz=-0.00226865106062467 -0.0340011106648613 0.0742813381426987 rpy=0.192483658660879 -0.0925172337475744 0.157672818669672
- joint right_finger5_joint2: axis -1 0 0 -> 0 1 0; limit lower=-0.37 upper=0.37 effort=0.1798 velocity=8.115781022 -> lower=-0.4203 upper=0.2931 effort=0.1798 velocity=8.1158; origin xyz=0.0022 0 0.004 rpy=0 0 0 -> xyz=0.0022000006995556 0 0.0040000052791524 rpy=0 0 1.5707963373693
- joint right_finger5_joint3: axis -0 1 -0 -> 0 1 0; limit lower=-0.4804 upper=1.5420 effort=0.2384 velocity=12.86307659 -> lower=-0.4804 upper=1.5420 effort=0.2384 velocity=12.863; origin xyz=-0.00475 0 0.043618 rpy=0 0 -0.00026861 -> xyz=0 0.00474999944502474 0.0436176874505066 rpy=0 0 -1.57106495008262
- joint right_finger5_joint4: axis -0 1 -0 -> 0 1 0; limit lower=-0.4705 upper=1.5709 effort=0.1866 velocity=13.57866158 -> lower=-0.4705 upper=1.5709 effort=0.1866 velocity=13.579; origin xyz=0 0 0.0295 rpy=0 0 0 -> xyz=0 -0.000200000003294461 0.0294999999999999 rpy=0 0 0
- joint right_finger5_tip_fixed: origin xyz=-0.0010446 1.1308E-05 0.0267 rpy=0 0 0 -> xyz=-0.00104463936847252 0.000211309529000607 0.0267000001662517 rpy=0 0 0

File: urdf/right.urdf (robot description, URDF)
Before this commit: robot wujihand-right, 26 links, 25 joints
Joints:
- joint right_finger1_joint1: axis -0 1 -0 -> 0 1 0; limit lower=0.0475 upper=1.6033 effort=0.4452 velocity=8.58701992 -> lower=0.0368 upper=1.6125 effort=0.4452 velocity=8.587; origin xyz=0.0085244 0.020575 0.028712 rpy=-1.328 -0.37161 -0.7307 -> xyz=0.0084398536891496 0.0205866432770798 0.0288928344360424 rpy=-1.32802443797267 -0.371613529401197 -0.730700470955738
- joint right_finger1_joint2: axis -0 -1 -0 -> 0 1 0; limit lower=-0.1387 upper=0.9324 effort=0.4259 velocity=11.10029404 -> lower=-0.1576 upper=0.9312 effort=0.4259 velocity=11.1; origin xyz=-0.0047549 -0.0060191 0.014132 rpy=-0.57428 -0.23677 1.8034 -> xyz=-0.00475489769909336 -0.00581913700106552 0.0141320977693281 rpy=0.574275025049342 0.236773483165491 -1.3381949894783
- joint right_finger1_joint3: limit lower=-0.4642 upper=1.5623 effort=0.1888 velocity=12.86307659 -> lower=-0.4638 upper=1.5607 effort=0.1888 velocity=12.863; origin xyz=0.00018873 -0.0009916 0.034664 rpy=0.049049 0.017311 -1.9085 -> xyz=-0.000266709908258896 0.000991501558320149 0.0346656189847898 rpy=0.0490494507279648 0.017311243665607 1.23305222676766
- joint right_finger1_joint4: limit lower=-0.4699 upper=1.5568 effort=0.1468 velocity=13.57866158 -> lower=-0.4829 upper=1.5451 effort=0.1468 velocity=13.578; origin xyz=0 -0.00025 0.0295 rpy=0 0 0 -> xyz=0 0.000200000007014398 0.0295000000021542 rpy=0 0 0
- joint right_finger1_tip_fixed: origin xyz=-0.0011048 0.00023218 0.0283 rpy=0 0 0 -> xyz=-0.00105000000124529 -0.000200000000000502 0.0272999999978436 rpy=0 0 0
- joint right_finger2_joint1: limit lower=-0.1585 upper=1.5604 effort=0.6188 velocity=8.203047484 -> lower=-0.1611 upper=1.5588 effort=0.6188 velocity=8.203; origin xyz=-0.0058701 0.029434 0.091917 rpy=-0.11071 -0.071139 -0.21822 -> xyz=-0.00587008921485247 0.0294338632809287 0.0919165306699325 rpy=-0.110709283985856 -0.0711392458057915 -0.218224846691839
- joint right_finger2_joint2: axis -1 0 0 -> 0 0.999999999978991 0; limit lower=-0.37 upper=0.37 effort=0.1822 velocity=8.115781022 -> lower=-0.4044 upper=0.3054 effort=0.1822 velocity=8.1158; origin xyz=0.0022 0 0.004 rpy=0 0 0 -> xyz=0.00220000016749383 0 0.00400000572323159 rpy=0 0 1.57079633736728
- joint right_finger2_joint3: axis -0 1 -0 -> 0 1 0; limit lower=-0.4777 upper=1.5485 effort=0.2251 velocity=12.86307659 -> lower=-0.4714 upper=1.5504 effort=0.2251 velocity=12.863; origin xyz=-0.0047503 0 0.043618 rpy=0 0 -0.00026861 -> xyz=0 0.00475028218260664 0.0436176566595782 rpy=0 0 -1.57106495008262
- joint right_finger2_joint4: axis -0 1 -0 -> 0 1 0; limit lower=-0.4683 upper=1.5753 effort=0.2170 velocity=13.57866158 -> lower=-0.4644 upper=1.5753 effort=0.2170 velocity=13.578; origin xyz=0 0 0.0295 rpy=0 0 0 -> xyz=0 -0.00020000000636031 0.0294999999999844 rpy=0 0 0
- joint right_finger2_tip_fixed: origin xyz=-0.00105 0 0.0274 rpy=0 0 0 -> xyz=-0.00104999999940632 0.000200000000000138 0.0266999989308851 rpy=0 0 0
- joint right_finger3_joint1: limit lower=-0.1644 upper=1.5516 effort=0.6494 velocity=8.203047484 -> lower=-0.1719 upper=1.5496 effort=0.6494 velocity=8.203; origin xyz=-0.01046 0.0074615 0.089544 rpy=-5.0886E-05 -0.087266 0.00058387 -> xyz=-0.0104597238611628 0.00746146014385576 0.0895435117703666 rpy=-5.08864726421373E-05 -0.0872664633653732 0.000583871740007801
- joint right_finger3_joint2: axis -1 0 0 -> 0 1 0; limit lower=-0.37 upper=0.37 effort=0.1827 velocity=8.115781022 -> lower=-0.4014 upper=0.2996 effort=0.1827 velocity=8.1158; origin xyz=0.0022 0 0.004 rpy=0 0 0 -> xyz=0.00220000049491006 0 0.00400000560544524 rpy=0 0 1.57079633736875
- joint right_finger3_joint3: axis -0 1 -0 -> 0 1 0; limit lower=-0.4739 upper=1.5512 effort=0.2078 velocity=12.86307659 -> lower=-0.4632 upper=1.5613 effort=0.2078 velocity=12.863; origin xyz=-0.00475 0 0.043618 rpy=0 0 -0.00026861 -> xyz=0 0.0047500001855858 0.0436176873657041 rpy=0 0 -1.57106495008262
- joint right_finger3_joint4: axis -0 1 -0 -> 0 1 0; limit lower=-0.4684 upper=1.5745 effort=0.2018 velocity=13.57866158 -> lower=-0.4697 upper=1.5702 effort=0.2018 velocity=13.579; origin xyz=0 0 0.0295 rpy=0 0 0 -> xyz=0 -0.000200000004070615 0.0294999999999999 rpy=0 0 0
- joint right_finger3_tip_fixed: origin xyz=-0.0010491 0 0.0267 rpy=0 0 0 -> xyz=-0.00104908716153243 0.000201039517772421 0.0266999998992792 rpy=0 0 0
- joint right_finger4_joint1: axis -0 1 -0 -> 0 1 0; limit lower=-0.1554 upper=1.5585 effort=0.6389 velocity=8.203047484 -> lower=-0.1601 upper=1.5534 effort=0.6389 velocity=8.203; origin xyz=-0.0076649 -0.013712 0.084429 rpy=0.090375 -0.083436 0.047127 -> xyz=-0.0076648599285041 -0.0137122383759844 0.084428694586379 rpy=0.0903746211775801 -0.0834355030065636 0.0471266290291302
- joint right_finger4_joint2: axis -1 0 0 -> 0 1 0; limit lower=-0.37 upper=0.37 effort=0.1832 velocity=8.115781022 -> lower=-0.4134 upper=0.3161 effort=0.1832 velocity=8.1158; origin xyz=0.0022 0 0.004 rpy=0 0 0 -> xyz=0.00220000052979842 0 0.00400000547923511 rpy=0 0 1.57079633736852
- joint right_finger4_joint3: axis -0 1 -0 -> 0 1 0; limit lower=-0.4765 upper=1.5487 effort=0.2249 velocity=12.86307659 -> lower=-0.4782 upper=1.5448 effort=0.2249 velocity=12.863; origin xyz=-0.00475 0 0.043618 rpy=0 0 -0.00026861 -> xyz=0 0.00474999949683786 0.0436176874505065 rpy=0 0 -1.57106495008262
- joint right_finger4_joint4: axis -0 1 -0 -> 0 1 0; limit lower=-0.4777 upper=1.5634 effort=0.2044 velocity=13.57866158 -> lower=-0.4825 upper=1.5550 effort=0.2044 velocity=13.579; origin xyz=0 0 0.0295 rpy=0 0 0 -> xyz=0 -0.000200000003294468 0.0294999999999999 rpy=0 0 0
- joint right_finger4_tip_fixed: origin xyz=-0.0010528 0 0.0267 rpy=0 0 0 -> xyz=-0.00105960974768627 0.000190450796499008 0.0266999999370233 rpy=0 0 0
- joint right_finger5_joint1: limit lower=-0.1626 upper=1.5585 effort=0.6441 velocity=8.203047484 -> lower=-0.1674 upper=1.5539 effort=0.6441 velocity=8.203; origin xyz=-0.0022687 -0.034001 0.074281 rpy=0.19248 -0.092517 0.15767 -> xyz=-0.00226865106062467 -0.0340011106648613 0.0742813381426987 rpy=0.192483658660879 -0.0925172337475744 0.157672818669672
- joint right_finger5_joint2: axis -1 0 0 -> 0 1 0; limit lower=-0.37 upper=0.37 effort=0.1798 velocity=8.115781022 -> lower=-0.4203 upper=0.2931 effort=0.1798 velocity=8.1158; origin xyz=0.0022 0 0.004 rpy=0 0 0 -> xyz=0.0022000006995556 0 0.0040000052791524 rpy=0 0 1.5707963373693
- joint right_finger5_joint3: axis -0 1 -0 -> 0 1 0; limit lower=-0.4768 upper=1.5490 effort=0.2384 velocity=12.86307659 -> lower=-0.4804 upper=1.5420 effort=0.2384 velocity=12.863; origin xyz=-0.00475 0 0.043618 rpy=0 0 -0.00026861 -> xyz=0 0.00474999944502474 0.0436176874505066 rpy=0 0 -1.57106495008262
- joint right_finger5_joint4: axis -0 1 -0 -> 0 1 0; limit lower=-0.4683 upper=1.5735 effort=0.1866 velocity=13.57866158 -> lower=-0.4705 upper=1.5709 effort=0.1866 velocity=13.579; origin xyz=0 0 0.0295 rpy=0 0 0 -> xyz=0 -0.000200000003294461 0.0294999999999999 rpy=0 0 0
- joint right_finger5_tip_fixed: origin xyz=-0.0010446 1.1308E-05 0.0267 rpy=0 0 0 -> xyz=-0.00104463936847252 0.000211309529000607 0.0267000001662517 rpy=0 0 0
