Commit message: fix: reverse axis for left finger3/finger4 joint2

File: urdf/left-ros.urdf (robot description, URDF)
Before this commit: robot wujihand-right-v1.0.2, 26 links, 25 joints
Joints:
- joint left_finger3_joint2: axis 1 0 0 -> -1 0 0
- joint left_finger4_joint2: axis 1 0 0 -> -1 0 0

File: urdf/left.urdf (robot description, URDF)
Before this commit: robot wujihand-right-v1.0.2, 26 links, 25 joints
Joints:
- joint left_finger3_joint2: axis 1 0 0 -> -1 0 0
- joint left_finger4_joint2: axis 1 0 0 -> -1 0 0

Commit message: fix: align MCP2 limits and release metadata

File: urdf/left-ros.urdf (robot description, URDF)
Before this commit: robot wujihand-left, 26 links, 25 joints
Joints:
- joint left_finger2_joint2: limit lower=-0.4095 upper=0.2921 effort=0.1822 velocity=8.115 -> lower=-0.37 upper=0.37 effort=0.1822 velocity=8.115
- joint left_finger3_joint2: limit lower=-0.3977 upper=0.3115 effort=0.1827 velocity=8.115 -> lower=-0.37 upper=0.37 effort=0.1827 velocity=8.115
- joint left_finger4_joint2: limit lower=-0.4101 upper=0.3014 effort=0.1832 velocity=8.115 -> lower=-0.37 upper=0.37 effort=0.1832 velocity=8.115
- joint left_finger5_joint2: limit lower=-0.4103 upper=0.2949 effort=0.1798 velocity=8.115 -> lower=-0.37 upper=0.37 effort=0.1798 velocity=8.115

File: urdf/left.urdf (robot description, URDF)
Before this commit: robot wujihand-left, 26 links, 25 joints
Joints:
- joint left_finger2_joint2: limit lower=-0.4069 upper=0.2988 effort=0.1822 velocity=8.115 -> lower=-0.37 upper=0.37 effort=0.1822 velocity=8.115
- joint left_finger3_joint2: limit lower=-0.3995 upper=0.3055 effort=0.1827 velocity=8.115 -> lower=-0.37 upper=0.37 effort=0.1827 velocity=8.115
- joint left_finger4_joint2: limit lower=-0.4118 upper=0.3087 effort=0.1832 velocity=8.115 -> lower=-0.37 upper=0.37 effort=0.1832 velocity=8.115
- joint left_finger5_joint2: limit lower=-0.4153 upper=0.2940 effort=0.1798 velocity=8.115 -> lower=-0.37 upper=0.37 effort=0.1798 velocity=8.115

File: urdf/right-ros.urdf (robot description, URDF)
Before this commit: robot wujihand-right, 26 links, 25 joints
Joints:
- joint right_finger2_joint2: limit lower=-0.4044 upper=0.3054 effort=0.1822 velocity=8.115781022 -> lower=-0.37 upper=0.37 effort=0.1822 velocity=8.115781022
- joint right_finger3_joint2: limit lower=-0.4014 upper=0.2996 effort=0.1827 velocity=8.115781022 -> lower=-0.37 upper=0.37 effort=0.1827 velocity=8.115781022
- joint right_finger4_joint2: limit lower=-0.4134 upper=0.3161 effort=0.1832 velocity=8.115781022 -> lower=-0.37 upper=0.37 effort=0.1832 velocity=8.115781022
- joint right_finger5_joint2: limit lower=-0.4203 upper=0.2931 effort=0.1798 velocity=8.115781022 -> lower=-0.37 upper=0.37 effort=0.1798 velocity=8.115781022

File: urdf/right.urdf (robot description, URDF)
Before this commit: robot wujihand-right, 26 links, 25 joints
Joints:
- joint right_finger2_joint2: limit lower=-0.4069 upper=0.2988 effort=0.1822 velocity=8.115781022 -> lower=-0.37 upper=0.37 effort=0.1822 velocity=8.115781022
- joint right_finger3_joint2: limit lower=-0.3995 upper=0.3055 effort=0.1827 velocity=8.115781022 -> lower=-0.37 upper=0.37 effort=0.1827 velocity=8.115781022
- joint right_finger4_joint2: limit lower=-0.4118 upper=0.3087 effort=0.1832 velocity=8.115781022 -> lower=-0.37 upper=0.37 effort=0.1832 velocity=8.115781022
- joint right_finger5_joint2: limit lower=-0.4153 upper=0.2940 effort=0.1798 velocity=8.115781022 -> lower=-0.37 upper=0.37 effort=0.1798 velocity=8.115781022
