Commit message: Release v1.0.0

File: urdf/left-ros.urdf (robot description, URDF)
Before this commit: robot wujihand-left, 26 links, 25 joints
Joints:
- joint left_finger1_joint1: axis 0 1 0 -> 0 -1 0; origin xyz=0.00843985365597852 -0.0205866432293554 0.0288928344107784 rpy=1.5023139401368 0.43577167910554 3.11264835810693 -> xyz=0.00843985365415843 -0.0205866432296062 0.0288928344146015 rpy=-1.32802443797267 0.371613529401196 -2.41089218263562
- joint left_finger1_joint2: axis 0 -1 0 -> 0 0.999999999999998 0; origin xyz=-0.0054483 0.0058191 -0.01388 rpy=0.14937 -0.34623 1.5901 -> xyz=0.00475489639781444 -0.00581913884095369 0.0141320959775981 rpy=-0.574275017658819 0.236773443835485 -1.80339762361133
- joint left_finger1_joint3: limit lower=-0.4646 upper=1.5639 effort=0.1888 velocity=13.578 -> lower=-0.4646 upper=1.5639 effort=0.1888 velocity=12.863; origin xyz=-0.000846961087777298 0.000991504133990267 -0.0346562987377679 rpy=0.0332538563601251 0.0117623260174173 -1.90877003040037 -> xyz=-0.000266710475105365 -0.000991501671842022 0.0346656206595102 rpy=-0.0490495013721327 0.0173112654625817 -1.23305223942119
- joint left_finger1_joint4: limit lower=-0.4570 upper=1.5684 effort=0.1468 velocity=12.863 -> lower=-0.4570 upper=1.5684 effort=0.1468 velocity=13.578; origin xyz=0 0 -0.0294999998969489 rpy=0 0 0 -> xyz=0 -0.000200000007014417 0.0294999998969491 rpy=0 0 0
- joint left_finger1_tip_fixed: origin xyz=0.00104999999999626 0 -0.0235000000000007 rpy=3.14159265358971 0 -3.14159265358979 -> xyz=-0.00104999999999688 0.000200000000001237 0.0272999999999996 rpy=0 0 0
- joint left_finger2_joint1: origin xyz=-0.00587008921400943 -0.0294338632807759 0.0919165306703557 rpy=0.110463316505378 -0.0251937198594477 0.223332069867641 -> xyz=-0.00587008921405553 -0.0294338632807666 0.0919165306703556 rpy=0.110709291859976 -0.0711392444947576 0.218224846837306
- joint left_finger2_joint2: axis -1 0 0 -> 0 1 0; limit lower=-0.37 upper=0.37 effort=0.1822 velocity=8.115 -> lower=-0.4095 upper=0.2921 effort=0.1822 velocity=8.115; origin xyz=0.000389540189408399 0 0.00402230398376657 rpy=0 -0.0462278050739338 0 -> xyz=0.00220000016133353 0 0.00400000572577126 rpy=0 0 1.57079631622159
- joint left_finger2_joint3: limit lower=-0.4839 upper=1.5466 effort=0.2251 velocity=13.578 -> lower=-0.4839 upper=1.5466 effort=0.2251 velocity=12.863; origin xyz=-0.00312502624735005 0.000100282455430194 0.0436176874512652 rpy=0 0 0.000268612717770449 -> xyz=0 0.00474999948522651 0.0436176874464638 rpy=0 0 -1.57052771407713
- joint left_finger2_joint4: limit lower=-0.4723 upper=1.5754 effort=0.2170 velocity=12.863 -> lower=-0.4723 upper=1.5754 effort=0.2170 velocity=13.578; origin xyz=0 0 0.0294999999999921 rpy=0 0 0 -> xyz=0 -0.00020000000114569 0.0295000000005511 rpy=0 0 0
- joint left_finger2_tip_fixed: origin xyz=-0.00199999998882132 -9.99999775618474E-05 0.0239466139626726 rpy=0 0 0 -> xyz=-0.00105210040162161 0.000210869249702341 0.0266999998503596 rpy=0 0 0
- joint left_finger3_joint1: origin xyz=-0.01046 -0.0074615 0.089544 rpy=5.0693E-05 0 -0.00057944 -> xyz=-0.0104597238646911 -0.00746146014383039 0.0895435117684639 rpy=5.08943582386716E-05 -0.0872664620461616 -0.000583871753342456
- joint left_finger3_joint2: axis -1 0 0 -> 0 1 0; limit lower=-0.37 upper=0.37 effort=0.1827 velocity=8.115 -> lower=-0.3977 upper=0.3115 effort=0.1827 velocity=8.115; origin xyz=0.000224188923157675 0 0.00403489896760838 rpy=0 -0.0872664630099629 0 -> xyz=0.00220000043882706 0 0.0040000056099367 rpy=0 0 1.57079631623283
- joint left_finger3_joint3: limit lower=-0.4847 upper=1.5411 effort=0.2078 velocity=13.578 -> lower=-0.4847 upper=1.5411 effort=0.2078 velocity=12.863; origin xyz=-0.00312502618421547 0.000100282625113788 0.0436176874508615 rpy=0 0 0.000268612717747223 -> xyz=0 0.00474999936719482 0.0436176874471427 rpy=0 0 -1.57052771407715
- joint left_finger3_joint4: limit lower=-0.4671 upper=1.5788 effort=0.2018 velocity=12.863 -> lower=-0.4671 upper=1.5788 effort=0.2018 velocity=13.578; origin xyz=0 0 0.0294999999999998 rpy=0 0 0 -> xyz=0 -0.000200000001145385 0.029499999999373 rpy=0 0 0
- joint left_finger3_tip_fixed: origin xyz=-0.00199999998882053 -9.99999999926624E-05 0.0239466139625789 rpy=0 0 0 -> xyz=-0.00105039969315103 0.000202672284305974 0.0266999998510997 rpy=0 0 0
- joint left_finger4_joint1: origin xyz=-0.0076649 0.013712 0.084429 rpy=-0.090059 0 -0.054679 -> xyz=-0.00766485992731566 0.0137122383759935 0.0844286945869771 rpy=-0.0903746132831303 -0.0834355016926537 -0.0471266291492555
- joint left_finger4_joint2: axis -1 0 0 -> 0 1 0; limit lower=-0.37 upper=0.37 effort=0.1832 velocity=8.115 -> lower=-0.4101 upper=0.3014 effort=0.1832 velocity=8.115; origin xyz=0.000238272023819444 0 0.00403409169489746 rpy=0 -0.0837758044893524 0 -> xyz=0.00220000046883515 0 0.00400000548163587 rpy=0 0 1.57079631622036
- joint left_finger4_joint3: limit lower=-0.4747 upper=1.5526 effort=0.2249 velocity=13.578 -> lower=-0.4747 upper=1.5526 effort=0.2249 velocity=12.863; origin xyz=-0.00312502629370909 0.000100282441161618 0.0436176874512648 rpy=0 0 0.000268623287696204 -> xyz=0 0.00474999947605386 0.0436176874464634 rpy=0 0 -1.5705277035072
- joint left_finger4_joint4: limit lower=-0.4729 upper=1.5718 effort=0.2044 velocity=12.863 -> lower=-0.4729 upper=1.5718 effort=0.2044 velocity=13.578; origin xyz=0 0 0.0295000000000005 rpy=0 0 0 -> xyz=0 -0.000200000001146229 0.0294999999999928 rpy=0 0 0
- joint left_finger4_tip_fixed: origin xyz=-0.00199999999999928 -9.99999794204474E-05 0.0239466139617312 rpy=0 0 0 -> xyz=-0.00104998290825126 0.000202557162358057 0.0266999998509249 rpy=0 0 0
- joint left_finger5_joint1: origin xyz=-0.00226865105948153 0.0340011106647822 0.0742813381432918 rpy=-0.191650218499317 0 -0.175676455157885 -> xyz=-0.00226865105942822 0.0340011106647859 0.0742813381432916 rpy=-0.192483650752976 -0.0925172324525506 -0.157672818923778
- joint left_finger5_joint2: axis -1 0 0 -> 0 1 0; limit lower=-0.37 upper=0.37 effort=0.1798 velocity=8.115 -> lower=-0.4103 upper=0.2949 effort=0.1798 velocity=8.115; origin xyz=0.000196015009673409 0 0.00403636545307588 rpy=0 -0.0942477800158131 0 -> xyz=0.0022000006386125 0 0.0040000052815589 rpy=0 0 1.57079631621958
- joint left_finger5_joint3: limit lower=-0.4733 upper=1.5560 effort=0.2384 velocity=13.578 -> lower=-0.4733 upper=1.5560 effort=0.2384 velocity=12.863; origin xyz=-0.00312502637316564 0.000100282626826854 0.0436176864544762 rpy=0 0 0.000268612717748753 -> xyz=0 0.00474999955614431 0.0436176864501152 rpy=0 0 -1.57052771407715
- joint left_finger5_joint4: limit lower=-0.4662 upper=1.5760 effort=0.1866 velocity=12.863 -> lower=-0.4662 upper=1.5760 effort=0.1866 velocity=13.578; origin xyz=0 0 0.0295000009963936 rpy=0 0 0 -> xyz=0 -0.000200000001688738 0.0295000009963858 rpy=0 0 0
- joint left_finger5_tip_fixed: origin xyz=-0.00200000001120192 -9.99999794204162E-05 0.0239466139607956 rpy=0 0 0 -> xyz=-0.00105040660537688 0.000201047212892366 0.0266999998509271 rpy=0 0 0

File: urdf/left.urdf (robot description, URDF)
Before this commit: robot wujihand-left, 26 links, 25 joints
Joints:
- joint left_finger1_joint1: axis 0 1 0 -> 0 -1 0; limit lower=0.0475 upper=1.6033 effort=0.4452 velocity=8.587 -> lower=0.0583 upper=1.5941 effort=0.4452 velocity=8.587; origin xyz=0.00843985365597852 -0.0205866432293554 0.0288928344107784 rpy=1.5023139401368 0.43577167910554 3.11264835810693 -> xyz=0.00843985365415843 -0.0205866432296062 0.0288928344146015 rpy=-1.32802443797267 0.371613529401196 -2.41089218263562
- joint left_finger1_joint2: axis 0 -1 0 -> 0 0.999999999999998 0; limit lower=-0.1387 upper=0.9324 effort=0.4259 velocity=11.1 -> lower=-0.1199 upper=0.9335 effort=0.4259 velocity=11.1; origin xyz=-0.0054483 0.0058191 -0.01388 rpy=0.14937 -0.34623 1.5901 -> xyz=0.00475489639781444 -0.00581913884095369 0.0141320959775981 rpy=-0.574275017658819 0.236773443835485 -1.80339762361133
- joint left_finger1_joint3: limit lower=-0.4642 upper=1.5623 effort=0.1888 velocity=13.578 -> lower=-0.4646 upper=1.5639 effort=0.1888 velocity=12.863; origin xyz=-0.000846961087777298 0.000991504133990267 -0.0346562987377679 rpy=0.0332538563601251 0.0117623260174173 -1.90877003040037 -> xyz=-0.000266710475105365 -0.000991501671842022 0.0346656206595102 rpy=-0.0490495013721327 0.0173112654625817 -1.23305223942119
- joint left_finger1_joint4: limit lower=-0.4699 upper=1.5568 effort=0.1468 velocity=12.863 -> lower=-0.4570 upper=1.5684 effort=0.1468 velocity=13.578; origin xyz=0 0 -0.0294999998969489 rpy=0 0 0 -> xyz=0 -0.000200000007014417 0.0294999998969491 rpy=0 0 0
- joint left_finger1_tip_fixed: origin xyz=0.00104999999999626 0 -0.0235000000000007 rpy=3.14159265358971 0 -3.14159265358979 -> xyz=-0.00104999999999688 0.000200000000001237 0.0272999999999996 rpy=0 0 0
- joint left_finger2_joint1: limit lower=-0.1585 upper=1.5604 effort=0.6188 velocity=8.203 -> lower=-0.1560 upper=1.5619 effort=0.6188 velocity=8.203; origin xyz=-0.00587008921400943 -0.0294338632807759 0.0919165306703557 rpy=0.110463316505378 -0.0251937198594477 0.223332069867641 -> xyz=-0.00587008921405553 -0.0294338632807666 0.0919165306703556 rpy=0.110709291859976 -0.0711392444947576 0.218224846837306
- joint left_finger2_joint2: axis -1 0 0 -> 0 1 0; limit lower=-0.37 upper=0.37 effort=0.1822 velocity=8.115 -> lower=-0.4095 upper=0.2921 effort=0.1822 velocity=8.115; origin xyz=0.000389540189408399 0 0.00402230398376657 rpy=0 -0.0462278050739338 0 -> xyz=0.00220000016133353 0 0.00400000572577126 rpy=0 0 1.57079631622159
- joint left_finger2_joint3: limit lower=-0.4777 upper=1.5485 effort=0.2251 velocity=13.578 -> lower=-0.4839 upper=1.5466 effort=0.2251 velocity=12.863; origin xyz=-0.00312502624735005 0.000100282455430194 0.0436176874512652 rpy=0 0 0.000268612717770449 -> xyz=0 0.00474999948522651 0.0436176874464638 rpy=0 0 -1.57052771407713
- joint left_finger2_joint4: limit lower=-0.4683 upper=1.5753 effort=0.2170 velocity=12.863 -> lower=-0.4723 upper=1.5754 effort=0.2170 velocity=13.578; origin xyz=0 0 0.0294999999999921 rpy=0 0 0 -> xyz=0 -0.00020000000114569 0.0295000000005511 rpy=0 0 0
- joint left_finger2_tip_fixed: origin xyz=-0.00199999998882132 -9.99999775618474E-05 0.0239466139626726 rpy=0 0 0 -> xyz=-0.00105210040162161 0.000210869249702341 0.0266999998503596 rpy=0 0 0
- joint left_finger3_joint1: limit lower=-0.1644 upper=1.5516 effort=0.6494 velocity=8.203 -> lower=-0.1569 upper=1.5536 effort=0.6494 velocity=8.203; origin xyz=-0.01046 -0.0074615 0.089544 rpy=5.0693E-05 0 -0.00057944 -> xyz=-0.0104597238646911 -0.00746146014383039 0.0895435117684639 rpy=5.08943582386716E-05 -0.0872664620461616 -0.000583871753342456
- joint left_finger3_joint2: axis -1 0 0 -> 0 1 0; limit lower=-0.37 upper=0.37 effort=0.1827 velocity=8.115 -> lower=-0.3977 upper=0.3115 effort=0.1827 velocity=8.115; origin xyz=0.000224188923157675 0 0.00403489896760838 rpy=0 -0.0872664630099629 0 -> xyz=0.00220000043882706 0 0.0040000056099367 rpy=0 0 1.57079631623283
- joint left_finger3_joint3: limit lower=-0.4739 upper=1.5512 effort=0.2078 velocity=13.578 -> lower=-0.4847 upper=1.5411 effort=0.2078 velocity=12.863; origin xyz=-0.00312502618421547 0.000100282625113788 0.0436176874508615 rpy=0 0 0.000268612717747223 -> xyz=0 0.00474999936719482 0.0436176874471427 rpy=0 0 -1.57052771407715
- joint left_finger3_joint4: limit lower=-0.4684 upper=1.5745 effort=0.2018 velocity=12.863 -> lower=-0.4671 upper=1.5788 effort=0.2018 velocity=13.578; origin xyz=0 0 0.0294999999999998 rpy=0 0 0 -> xyz=0 -0.000200000001145385 0.029499999999373 rpy=0 0 0
- joint left_finger3_tip_fixed: origin xyz=-0.00199999998882053 -9.99999999926624E-05 0.0239466139625789 rpy=0 0 0 -> xyz=-0.00105039969315103 0.000202672284305974 0.0266999998510997 rpy=0 0 0
- joint left_finger4_joint1: limit lower=-0.1554 upper=1.5585 effort=0.6389 velocity=8.203 -> lower=-0.1507 upper=1.5636 effort=0.6389 velocity=8.203; origin xyz=-0.0076649 0.013712 0.084429 rpy=-0.090059 0 -0.054679 -> xyz=-0.00766485992731566 0.0137122383759935 0.0844286945869771 rpy=-0.0903746132831303 -0.0834355016926537 -0.0471266291492555
- joint left_finger4_joint2: axis -1 0 0 -> 0 1 0; limit lower=-0.37 upper=0.37 effort=0.1832 velocity=8.115 -> lower=-0.4101 upper=0.3014 effort=0.1832 velocity=8.115; origin xyz=0.000238272023819444 0 0.00403409169489746 rpy=0 -0.0837758044893524 0 -> xyz=0.00220000046883515 0 0.00400000548163587 rpy=0 0 1.57079631622036
- joint left_finger4_joint3: limit lower=-0.4765 upper=1.5487 effort=0.2249 velocity=13.578 -> lower=-0.4747 upper=1.5526 effort=0.2249 velocity=12.863; origin xyz=-0.00312502629370909 0.000100282441161618 0.0436176874512648 rpy=0 0 0.000268623287696204 -> xyz=0 0.00474999947605386 0.0436176874464634 rpy=0 0 -1.5705277035072
- joint left_finger4_joint4: limit lower=-0.4777 upper=1.5634 effort=0.2044 velocity=12.863 -> lower=-0.4729 upper=1.5718 effort=0.2044 velocity=13.578; origin xyz=0 0 0.0295000000000005 rpy=0 0 0 -> xyz=0 -0.000200000001146229 0.0294999999999928 rpy=0 0 0
- joint left_finger4_tip_fixed: origin xyz=-0.00199999999999928 -9.99999794204474E-05 0.0239466139617312 rpy=0 0 0 -> xyz=-0.00104998290825126 0.000202557162358057 0.0266999998509249 rpy=0 0 0
- joint left_finger5_joint1: limit lower=-0.1626 upper=1.5585 effort=0.6441 velocity=8.203 -> lower=-0.1578 upper=1.5632 effort=0.6441 velocity=8.203; origin xyz=-0.00226865105948153 0.0340011106647822 0.0742813381432918 rpy=-0.191650218499317 0 -0.175676455157885 -> xyz=-0.00226865105942822 0.0340011106647859 0.0742813381432916 rpy=-0.192483650752976 -0.0925172324525506 -0.157672818923778
- joint left_finger5_joint2: axis -1 0 0 -> 0 1 0; limit lower=-0.37 upper=0.37 effort=0.1798 velocity=8.115 -> lower=-0.4103 upper=0.2949 effort=0.1798 velocity=8.115; origin xyz=0.000196015009673409 0 0.00403636545307588 rpy=0 -0.0942477800158131 0 -> xyz=0.0022000006386125 0 0.0040000052815589 rpy=0 0 1.57079631621958
- joint left_finger5_joint3: limit lower=-0.4768 upper=1.5490 effort=0.2384 velocity=13.578 -> lower=-0.4733 upper=1.5560 effort=0.2384 velocity=12.863; origin xyz=-0.00312502637316564 0.000100282626826854 0.0436176864544762 rpy=0 0 0.000268612717748753 -> xyz=0 0.00474999955614431 0.0436176864501152 rpy=0 0 -1.57052771407715
- joint left_finger5_joint4: limit lower=-0.4683 upper=1.5735 effort=0.1866 velocity=12.863 -> lower=-0.4662 upper=1.5760 effort=0.1866 velocity=13.578; origin xyz=0 0 0.0295000009963936 rpy=0 0 0 -> xyz=0 -0.000200000001688738 0.0295000009963858 rpy=0 0 0
- joint left_finger5_tip_fixed: origin xyz=-0.00200000001120192 -9.99999794204162E-05 0.0239466139607956 rpy=0 0 0 -> xyz=-0.00105040660537688 0.000201047212892366 0.0266999998509271 rpy=0 0 0

File: urdf/right-ros.urdf (robot description, URDF)
Before this commit: robot wujihand-right, 26 links, 25 joints
Joints:
- joint right_finger1_joint1: axis -0 1 -0 -> 0 1 0; limit lower=0.0368 upper=1.6125 effort=0.4452 velocity=8.58701992 -> lower=0.0368 upper=1.6125 effort=0.4452 velocity=8.587; origin xyz=0.0085244 0.020575 0.028712 rpy=-1.328 -0.37161 -0.7307 -> xyz=0.0084398536891496 0.0205866432770798 0.0288928344360424 rpy=-1.32802443797267 -0.371613529401197 -0.730700470955738
- joint right_finger1_joint2: axis -0 -1 -0 -> 0 1 0; limit lower=-0.1576 upper=0.9312 effort=0.4259 velocity=11.10029404 -> lower=-0.1576 upper=0.9312 effort=0.4259 velocity=11.1; origin xyz=-0.0047549 -0.0060191 0.014132 rpy=-0.57428 -0.23677 1.8034 -> xyz=-0.00475489769909336 -0.00581913700106552 0.0141320977693281 rpy=0.574275025049342 0.236773483165491 -1.3381949894783
- joint right_finger1_joint3: limit lower=-0.4638 upper=1.5607 effort=0.1888 velocity=12.86307659 -> lower=-0.4638 upper=1.5607 effort=0.1888 velocity=12.863; origin xyz=0.00018873 -0.0009916 0.034664 rpy=0.049049 0.017311 -1.9085 -> xyz=-0.000266709908258896 0.000991501558320149 0.0346656189847898 rpy=0.0490494507279648 0.017311243665607 1.23305222676766
- joint right_finger1_joint4: limit lower=-0.4829 upper=1.5451 effort=0.1468 velocity=13.57866158 -> lower=-0.4829 upper=1.5451 effort=0.1468 velocity=13.578; origin xyz=0 -0.00025 0.0295 rpy=0 0 0 -> xyz=0 0.000200000007014398 0.0295000000021542 rpy=0 0 0
- joint right_finger1_tip_fixed: limit (none) -> lower=0 upper=0 effort=100 velocity=10; origin xyz=-0.0011048 0.00023218 0.0283 rpy=0 0 0 -> xyz=-0.00105000000124529 -0.000200000000000502 0.0272999999978436 rpy=0 0 0
- joint right_finger2_joint1: limit lower=-0.1611 upper=1.5588 effort=0.6188 velocity=8.203047484 -> lower=-0.1611 upper=1.5588 effort=0.6188 velocity=8.203; origin xyz=-0.0058701 0.029434 0.091917 rpy=-0.11071 -0.071139 -0.21822 -> xyz=-0.00587008921485247 0.0294338632809287 0.0919165306699325 rpy=-0.110709283985856 -0.0711392458057915 -0.218224846691839
- joint right_finger2_joint2: axis -1 0 0 -> 0 0.999999999978991 0; limit lower=-0.37 upper=0.37 effort=0.1822 velocity=8.115781022 -> lower=-0.4044 upper=0.3054 effort=0.1822 velocity=8.1158; origin xyz=0.0022 0 0.004 rpy=0 0 0 -> xyz=0.00220000016749383 0 0.00400000572323159 rpy=0 0 1.57079633736728
- joint right_finger2_joint3: axis -0 1 -0 -> 0 1 0; limit lower=-0.4714 upper=1.5504 effort=0.2251 velocity=12.86307659 -> lower=-0.4714 upper=1.5504 effort=0.2251 velocity=12.863; origin xyz=-0.0047503 0 0.043618 rpy=0 0 -0.00026861 -> xyz=0 0.00475028218260664 0.0436176566595782 rpy=0 0 -1.57106495008262
- joint right_finger2_joint4: axis -0 1 -0 -> 0 1 0; limit lower=-0.4644 upper=1.5753 effort=0.2170 velocity=13.57866158 -> lower=-0.4644 upper=1.5753 effort=0.2170 velocity=13.578; origin xyz=0 0 0.0295 rpy=0 0 0 -> xyz=0 -0.00020000000636031 0.0294999999999844 rpy=0 0 0
- joint right_finger2_tip_fixed: limit (none) -> lower=0 upper=0 effort=100 velocity=10; origin xyz=-0.00105 0 0.0274 rpy=0 0 0 -> xyz=-0.00104999999940632 0.000200000000000138 0.0266999989308851 rpy=0 0 0
- joint right_finger3_joint1: limit lower=-0.1719 upper=1.5496 effort=0.6494 velocity=8.203047484 -> lower=-0.1719 upper=1.5496 effort=0.6494 velocity=8.203; origin xyz=-0.01046 0.0074615 0.089544 rpy=-5.0886E-05 -0.087266 0.00058387 -> xyz=-0.0104597238611628 0.00746146014385576 0.0895435117703666 rpy=-5.08864726421373E-05 -0.0872664633653732 0.000583871740007801
- joint right_finger3_joint2: axis -1 0 0 -> 0 1 0; limit lower=-0.37 upper=0.37 effort=0.1827 velocity=8.115781022 -> lower=-0.4014 upper=0.2996 effort=0.1827 velocity=8.1158; origin xyz=0.0022 0 0.004 rpy=0 0 0 -> xyz=0.00220000049491006 0 0.00400000560544524 rpy=0 0 1.57079633736875
- joint right_finger3_joint3: axis -0 1 -0 -> 0 1 0; limit lower=-0.4632 upper=1.5613 effort=0.2078 velocity=12.86307659 -> lower=-0.4632 upper=1.5613 effort=0.2078 velocity=12.863; origin xyz=-0.00475 0 0.043618 rpy=0 0 -0.00026861 -> xyz=0 0.0047500001855858 0.0436176873657041 rpy=0 0 -1.57106495008262
- joint right_finger3_joint4: axis -0 1 -0 -> 0 1 0; limit lower=-0.4697 upper=1.5702 effort=0.2018 velocity=13.57866158 -> lower=-0.4697 upper=1.5702 effort=0.2018 velocity=13.579; origin xyz=0 0 0.0295 rpy=0 0 0 -> xyz=0 -0.000200000004070615 0.0294999999999999 rpy=0 0 0
- joint right_finger3_tip_fixed: limit (none) -> lower=0 upper=0 effort=100 velocity=10; origin xyz=-0.0010491 0 0.0267 rpy=0 0 0 -> xyz=-0.00104908716153243 0.000201039517772421 0.0266999998992792 rpy=0 0 0
- joint right_finger4_joint1: axis -0 1 -0 -> 0 1 0; limit lower=-0.1601 upper=1.5534 effort=0.6389 velocity=8.203047484 -> lower=-0.1601 upper=1.5534 effort=0.6389 velocity=8.203; origin xyz=-0.0076649 -0.013712 0.084429 rpy=0.090375 -0.083436 0.047127 -> xyz=-0.0076648599285041 -0.0137122383759844 0.084428694586379 rpy=0.0903746211775801 -0.0834355030065636 0.0471266290291302
- joint right_finger4_joint2: axis -1 0 0 -> 0 1 0; limit lower=-0.37 upper=0.37 effort=0.1832 velocity=8.115781022 -> lower=-0.4134 upper=0.3161 effort=0.1832 velocity=8.1158; origin xyz=0.0022 0 0.004 rpy=0 0 0 -> xyz=0.00220000052979842 0 0.00400000547923511 rpy=0 0 1.57079633736852
- joint right_finger4_joint3: axis -0 1 -0 -> 0 1 0; limit lower=-0.4782 upper=1.5448 effort=0.2249 velocity=12.86307659 -> lower=-0.4782 upper=1.5448 effort=0.2249 velocity=12.863; origin xyz=-0.00475 0 0.043618 rpy=0 0 -0.00026861 -> xyz=0 0.00474999949683786 0.0436176874505065 rpy=0 0 -1.57106495008262
- joint right_finger4_joint4: axis -0 1 -0 -> 0 1 0; limit lower=-0.4825 upper=1.5550 effort=0.2044 velocity=13.57866158 -> lower=-0.4825 upper=1.5550 effort=0.2044 velocity=13.579; origin xyz=0 0 0.0295 rpy=0 0 0 -> xyz=0 -0.000200000003294468 0.0294999999999999 rpy=0 0 0
- joint right_finger4_tip_fixed: limit (none) -> lower=0 upper=0 effort=100 velocity=10; origin xyz=-0.0010528 0 0.0267 rpy=0 0 0 -> xyz=-0.00105960974768627 0.000190450796499008 0.0266999999370233 rpy=0 0 0
- joint right_finger5_joint1: limit lower=-0.1674 upper=1.5539 effort=0.6441 velocity=8.203047484 -> lower=-0.1674 upper=1.5539 effort=0.6441 velocity=8.203; origin xyz=-0.0022687 -0.034001 0.074281 rpy=0.19248 -0.092517 0.15767 -> xyz=-0.00226865106062467 -0.0340011106648613 0.0742813381426987 rpy=0.192483658660879 -0.0925172337475744 0.157672818669672
- joint right_finger5_joint2: axis -1 0 0 -> 0 1 0; limit lower=-0.37 upper=0.37 effort=0.1798 velocity=8.115781022 -> lower=-0.4203 upper=0.2931 effort=0.1798 velocity=8.1158; origin xyz=0.0022 0 0.004 rpy=0 0 0 -> xyz=0.0022000006995556 0 0.0040000052791524 rpy=0 0 1.5707963373693
- joint right_finger5_joint3: axis -0 1 -0 -> 0 1 0; limit lower=-0.4804 upper=1.5420 effort=0.2384 velocity=12.86307659 -> lower=-0.4804 upper=1.5420 effort=0.2384 velocity=12.863; origin xyz=-0.00475 0 0.043618 rpy=0 0 -0.00026861 -> xyz=0 0.00474999944502474 0.0436176874505066 rpy=0 0 -1.57106495008262
- joint right_finger5_joint4: axis -0 1 -0 -> 0 1 0; limit lower=-0.4705 upper=1.5709 effort=0.1866 velocity=13.57866158 -> lower=-0.4705 upper=1.5709 effort=0.1866 velocity=13.579; origin xyz=0 0 0.0295 rpy=0 0 0 -> xyz=0 -0.000200000003294461 0.0294999999999999 rpy=0 0 0
- joint right_finger5_tip_fixed: limit (none) -> lower=0 upper=0 effort=100 velocity=10; origin xyz=-0.0010446 1.1308E-05 0.0267 rpy=0 0 0 -> xyz=-0.00104463936847252 0.000211309529000607 0.0267000001662517 rpy=0 0 0
