Commit message: fix: thumb mesh vertices on both hands
Update thumb (finger1) STL meshes and sync URDF/MJCF/USD to match.
This batch also rolls up several regressions picked up from the
upstream urdf_cali pipeline:

- Restore left_finger5_link1 inertial xyz and material rgba in
  urdf/left.urdf and urdf/left-ros.urdf (both had decayed to URDF
  spec defaults: 0 0 0 and 1 1 1 1). Also patch the corresponding
  zeroed COM in usd/left/configuration/wujihand_physics.usd.
- Clamp 8 MJCF actuator ctrlrange upper bounds back within their
  joint range (same root cause as PR #33 hotfix: the 3-decimal
  export rounded above the 4-decimal joint range).
- Restore <mujoco><compiler .../></mujoco> block in all four URDFs
  for direct mujoco.MjModel.from_xml_path() loading.
- Align MJCF joint range values with the URDF unified limits
  (extends PR #36 unification into MJCF).
- Normalize URDF numeric precision to 7 significant digits across
  origin xyz/rpy, inertia, mass, and rgba.

File: urdf/left-ros.urdf (robot description, URDF)
Before this commit: robot wujihand-left, 26 links, 25 joints
Joints:
- joint left_finger1_joint1: axis 0 -1 0 -> 0 1 0; origin xyz=0.00843985365415843 -0.0205866432296062 0.0288928344146015 rpy=-1.32802443797267 0.371613529401196 -2.41089218263562 -> xyz=0.0084399 -0.020587 0.028893 rpy=1.328 -0.37161 0.7307
- joint left_finger1_joint2: axis 0 0.999999999999998 0 -> 0 -1 0; origin xyz=0.00475489639781444 -0.00581913884095369 0.0141320959775981 rpy=-0.574275017658819 0.236773443835485 -1.80339762361133 -> xyz=-0.0047549 0.0058191 0.014132 rpy=0.57428 -0.23677 -1.8034
- joint left_finger1_joint3: origin xyz=-0.000266710475105365 -0.000991501671842022 0.0346656206595102 rpy=-0.0490495013721327 0.0173112654625817 -1.23305223942119 -> xyz=0.00026671 0.0009915 0.034666 rpy=-0.049049 0.017311 1.9085
- joint left_finger1_joint4: origin xyz=0 -0.000200000007014417 0.0294999998969491 rpy=0 0 0 -> xyz=0 -0.0002 0.0295 rpy=0 0 0
- joint left_finger1_tip_fixed: axis 0 0 0 -> (none); origin xyz=-0.00104999999999688 0.000200000000001237 0.0272999999999996 rpy=0 0 0 -> xyz=-0.00105 0.0002 0.0313 rpy=0 0 0
- joint left_finger2_joint1: origin xyz=-0.00587008921405553 -0.0294338632807666 0.0919165306703556 rpy=0.110709291859976 -0.0711392444947576 0.218224846837306 -> xyz=-0.0058701 -0.029434 0.091917 rpy=0.11071 -0.071139 0.21822
- joint left_finger2_joint2: limit lower=-0.37 upper=0.37 effort=0.1822 velocity=8.115 -> lower=-0.3700 upper=0.3700 effort=0.1822 velocity=8.115; origin xyz=0.00220000016133353 0 0.00400000572577126 rpy=0 0 1.57079631622159 -> xyz=0.0022 0 0.004000006 rpy=0 0 1.570796
- joint left_finger2_joint3: origin xyz=0 0.00474999948522651 0.0436176874464638 rpy=0 0 -1.57052771407713 -> xyz=0 0.004749999 0.04361769 rpy=0 0 -1.570528
- joint left_finger2_joint4: origin xyz=0 -0.00020000000114569 0.0295000000005511 rpy=0 0 0 -> xyz=0 -0.0002 0.0295 rpy=0 0 0
- joint left_finger2_tip_fixed: axis 0 0 0 -> (none); origin xyz=-0.00105210040162161 0.000210869249702341 0.0266999998503596 rpy=0 0 0 -> xyz=-0.0010521 0.0002108692 0.0267 rpy=0 0 0
- joint left_finger3_joint1: origin xyz=-0.0104597238646911 -0.00746146014383039 0.0895435117684639 rpy=5.08943582386716E-05 -0.0872664620461616 -0.000583871753342456 -> xyz=-0.01046 -0.0074615 0.089544 rpy=5.0894e-05 -0.087266 -0.00058387
- joint left_finger3_joint2: limit lower=-0.37 upper=0.37 effort=0.1827 velocity=8.115 -> lower=-0.3700 upper=0.3700 effort=0.1827 velocity=8.115; origin xyz=0.00220000043882706 0 0.0040000056099367 rpy=0 0 1.57079631623283 -> xyz=0.0022 0 0.004000006 rpy=0 0 1.570796
- joint left_finger3_joint3: origin xyz=0 0.00474999936719482 0.0436176874471427 rpy=0 0 -1.57052771407715 -> xyz=0 0.004749999 0.04361769 rpy=0 0 -1.570528
- joint left_finger3_joint4: origin xyz=0 -0.000200000001145385 0.029499999999373 rpy=0 0 0 -> xyz=0 -0.0002 0.0295 rpy=0 0 0
- joint left_finger3_tip_fixed: axis 0 0 0 -> (none); origin xyz=-0.00105039969315103 0.000202672284305974 0.0266999998510997 rpy=0 0 0 -> xyz=-0.0010504 0.0002026723 0.0267 rpy=0 0 0
- joint left_finger4_joint1: origin xyz=-0.00766485992731566 0.0137122383759935 0.0844286945869771 rpy=-0.0903746132831303 -0.0834355016926537 -0.0471266291492555 -> xyz=-0.0076649 0.013712 0.084429 rpy=-0.090375 -0.083436 -0.047127
- joint left_finger4_joint2: limit lower=-0.37 upper=0.37 effort=0.1832 velocity=8.115 -> lower=-0.3700 upper=0.3700 effort=0.1832 velocity=8.115; origin xyz=0.00220000046883515 0 0.00400000548163587 rpy=0 0 1.57079631622036 -> xyz=0.0022 0 0.004000005 rpy=0 0 1.570796
- joint left_finger4_joint3: origin xyz=0 0.00474999947605386 0.0436176874464634 rpy=0 0 -1.5705277035072 -> xyz=0 0.004749999 0.04361769 rpy=0 0 -1.570528
- joint left_finger4_joint4: origin xyz=0 -0.000200000001146229 0.0294999999999928 rpy=0 0 0 -> xyz=0 -0.0002 0.0295 rpy=0 0 0
- joint left_finger4_tip_fixed: axis 0 0 0 -> (none); origin xyz=-0.00104998290825126 0.000202557162358057 0.0266999998509249 rpy=0 0 0 -> xyz=-0.001049983 0.0002025572 0.0267 rpy=0 0 0
- joint left_finger5_joint1: origin xyz=-0.00226865105942822 0.0340011106647859 0.0742813381432916 rpy=-0.192483650752976 -0.0925172324525506 -0.157672818923778 -> xyz=-0.002268651 0.03400111 0.07428134 rpy=-0.1924837 -0.09251723 -0.1576728
- joint left_finger5_joint2: limit lower=-0.37 upper=0.37 effort=0.1798 velocity=8.115 -> lower=-0.3700 upper=0.3700 effort=0.1798 velocity=8.115; origin xyz=0.0022000006386125 0 0.0040000052815589 rpy=0 0 1.57079631621958 -> xyz=0.002200001 0 0.004000005 rpy=0 0 1.570796
- joint left_finger5_joint3: origin xyz=0 0.00474999955614431 0.0436176864501152 rpy=0 0 -1.57052771407715 -> xyz=0 0.00475 0.04361769 rpy=0 0 -1.570528
- joint left_finger5_joint4: origin xyz=0 -0.000200000001688738 0.0295000009963858 rpy=0 0 0 -> xyz=0 -0.0002 0.0295 rpy=0 0 0
- joint left_finger5_tip_fixed: axis 0 0 0 -> (none); origin xyz=-0.00105040660537688 0.000201047212892366 0.0266999998509271 rpy=0 0 0 -> xyz=-0.001050407 0.0002010472 0.0267 rpy=0 0 0

File: urdf/left.urdf (robot description, URDF)
Before this commit: robot wujihand-left, 26 links, 25 joints
Joints:
- joint left_finger1_joint1: axis 0 -1 0 -> 0 1 0; origin xyz=0.00843985365415843 -0.0205866432296062 0.0288928344146015 rpy=-1.32802443797267 0.371613529401196 -2.41089218263562 -> xyz=0.0084399 -0.020587 0.028893 rpy=1.328 -0.37161 0.7307
- joint left_finger1_joint2: axis 0 0.999999999999998 0 -> 0 -1 0; origin xyz=0.00475489639781444 -0.00581913884095369 0.0141320959775981 rpy=-0.574275017658819 0.236773443835485 -1.80339762361133 -> xyz=-0.0047549 0.0058191 0.014132 rpy=0.57428 -0.23677 -1.8034
- joint left_finger1_joint3: origin xyz=-0.000266710475105365 -0.000991501671842022 0.0346656206595102 rpy=-0.0490495013721327 0.0173112654625817 -1.23305223942119 -> xyz=0.00026671 0.0009915 0.034666 rpy=-0.049049 0.017311 1.9085
- joint left_finger1_joint4: origin xyz=0 -0.000200000007014417 0.0294999998969491 rpy=0 0 0 -> xyz=0 -0.0002 0.0295 rpy=0 0 0
- joint left_finger1_tip_fixed: axis 0 0 0 -> (none); origin xyz=-0.00104999999999688 0.000200000000001237 0.0272999999999996 rpy=0 0 0 -> xyz=-0.00105 0.0002 0.0313 rpy=0 0 0
- joint left_finger2_joint1: origin xyz=-0.00587008921405553 -0.0294338632807666 0.0919165306703556 rpy=0.110709291859976 -0.0711392444947576 0.218224846837306 -> xyz=-0.0058701 -0.029434 0.091917 rpy=0.11071 -0.071139 0.21822
- joint left_finger2_joint2: limit lower=-0.37 upper=0.37 effort=0.1822 velocity=8.115 -> lower=-0.3700 upper=0.3700 effort=0.1822 velocity=8.115; origin xyz=0.00220000016133353 0 0.00400000572577126 rpy=0 0 1.57079631622159 -> xyz=0.0022 0 0.004000006 rpy=0 0 1.570796
- joint left_finger2_joint3: origin xyz=0 0.00474999948522651 0.0436176874464638 rpy=0 0 -1.57052771407713 -> xyz=0 0.004749999 0.04361769 rpy=0 0 -1.570528
- joint left_finger2_joint4: origin xyz=0 -0.00020000000114569 0.0295000000005511 rpy=0 0 0 -> xyz=0 -0.0002 0.0295 rpy=0 0 0
- joint left_finger2_tip_fixed: axis 0 0 0 -> (none); origin xyz=-0.00105210040162161 0.000210869249702341 0.0266999998503596 rpy=0 0 0 -> xyz=-0.0010521 0.0002108692 0.0267 rpy=0 0 0
- joint left_finger3_joint1: origin xyz=-0.0104597238646911 -0.00746146014383039 0.0895435117684639 rpy=5.08943582386716E-05 -0.0872664620461616 -0.000583871753342456 -> xyz=-0.01046 -0.0074615 0.089544 rpy=5.0894e-05 -0.087266 -0.00058387
- joint left_finger3_joint2: limit lower=-0.37 upper=0.37 effort=0.1827 velocity=8.115 -> lower=-0.3700 upper=0.3700 effort=0.1827 velocity=8.115; origin xyz=0.00220000043882706 0 0.0040000056099367 rpy=0 0 1.57079631623283 -> xyz=0.0022 0 0.004000006 rpy=0 0 1.570796
- joint left_finger3_joint3: origin xyz=0 0.00474999936719482 0.0436176874471427 rpy=0 0 -1.57052771407715 -> xyz=0 0.004749999 0.04361769 rpy=0 0 -1.570528
- joint left_finger3_joint4: origin xyz=0 -0.000200000001145385 0.029499999999373 rpy=0 0 0 -> xyz=0 -0.0002 0.0295 rpy=0 0 0
- joint left_finger3_tip_fixed: axis 0 0 0 -> (none); origin xyz=-0.00105039969315103 0.000202672284305974 0.0266999998510997 rpy=0 0 0 -> xyz=-0.0010504 0.0002026723 0.0267 rpy=0 0 0
- joint left_finger4_joint1: origin xyz=-0.00766485992731566 0.0137122383759935 0.0844286945869771 rpy=-0.0903746132831303 -0.0834355016926537 -0.0471266291492555 -> xyz=-0.0076649 0.013712 0.084429 rpy=-0.090375 -0.083436 -0.047127
- joint left_finger4_joint2: limit lower=-0.37 upper=0.37 effort=0.1832 velocity=8.115 -> lower=-0.3700 upper=0.3700 effort=0.1832 velocity=8.115; origin xyz=0.00220000046883515 0 0.00400000548163587 rpy=0 0 1.57079631622036 -> xyz=0.0022 0 0.004000005 rpy=0 0 1.570796
- joint left_finger4_joint3: origin xyz=0 0.00474999947605386 0.0436176874464634 rpy=0 0 -1.5705277035072 -> xyz=0 0.004749999 0.04361769 rpy=0 0 -1.570528
- joint left_finger4_joint4: origin xyz=0 -0.000200000001146229 0.0294999999999928 rpy=0 0 0 -> xyz=0 -0.0002 0.0295 rpy=0 0 0
- joint left_finger4_tip_fixed: axis 0 0 0 -> (none); origin xyz=-0.00104998290825126 0.000202557162358057 0.0266999998509249 rpy=0 0 0 -> xyz=-0.001049983 0.0002025572 0.0267 rpy=0 0 0
- joint left_finger5_joint1: origin xyz=-0.00226865105942822 0.0340011106647859 0.0742813381432916 rpy=-0.192483650752976 -0.0925172324525506 -0.157672818923778 -> xyz=-0.002268651 0.03400111 0.07428134 rpy=-0.1924837 -0.09251723 -0.1576728
- joint left_finger5_joint2: limit lower=-0.37 upper=0.37 effort=0.1798 velocity=8.115 -> lower=-0.3700 upper=0.3700 effort=0.1798 velocity=8.115; origin xyz=0.0022000006386125 0 0.0040000052815589 rpy=0 0 1.57079631621958 -> xyz=0.002200001 0 0.004000005 rpy=0 0 1.570796
- joint left_finger5_joint3: origin xyz=0 0.00474999955614431 0.0436176864501152 rpy=0 0 -1.57052771407715 -> xyz=0 0.00475 0.04361769 rpy=0 0 -1.570528
- joint left_finger5_joint4: origin xyz=0 -0.000200000001688738 0.0295000009963858 rpy=0 0 0 -> xyz=0 -0.0002 0.0295 rpy=0 0 0
- joint left_finger5_tip_fixed: axis 0 0 0 -> (none); origin xyz=-0.00105040660537688 0.000201047212892366 0.0266999998509271 rpy=0 0 0 -> xyz=-0.001050407 0.0002010472 0.0267 rpy=0 0 0

File: urdf/right-ros.urdf (robot description, URDF)
Before this commit: robot wujihand-right, 26 links, 25 joints
Joints:
- joint right_finger1_joint1: origin xyz=0.0084398536891496 0.0205866432770798 0.0288928344360424 rpy=-1.32802443797267 -0.371613529401197 -0.730700470955738 -> xyz=0.0084399 0.020587 0.028893 rpy=-1.328 -0.37161 -0.7307
- joint right_finger1_joint2: origin xyz=-0.00475489769909336 -0.00581913700106552 0.0141320977693281 rpy=0.574275025049342 0.236773483165491 -1.3381949894783 -> xyz=-0.0047549 -0.0058191 0.014132 rpy=0.57428 0.23677 -1.3382
- joint right_finger1_joint3: origin xyz=-0.000266709908258896 0.000991501558320149 0.0346656189847898 rpy=0.0490494507279648 0.017311243665607 1.23305222676766 -> xyz=-0.000266705 0.0009915016 0.03466562 rpy=0.04904945 0.01731124 1.233052
- joint right_finger1_joint4: origin xyz=0 0.000200000007014398 0.0295000000021542 rpy=0 0 0 -> xyz=0 0.0002 0.0295 rpy=0 0 0
- joint right_finger1_tip_fixed: axis 0 0 0 -> (none); origin xyz=-0.00105000000124529 -0.000200000000000502 0.0272999999978436 rpy=0 0 0 -> xyz=-0.00105 -0.0002 0.0313 rpy=0 0 0
- joint right_finger2_joint1: origin xyz=-0.00587008921485247 0.0294338632809287 0.0919165306699325 rpy=-0.110709283985856 -0.0711392458057915 -0.218224846691839 -> xyz=-0.0058701 0.029434 0.091917 rpy=-0.11071 -0.071139 -0.21822
- joint right_finger2_joint2: axis 0 0.999999999978991 0 -> 0 1 0; limit lower=-0.37 upper=0.37 effort=0.1822 velocity=8.1158 -> lower=-0.3700 upper=0.3700 effort=0.1822 velocity=8.115; origin xyz=0.00220000016749383 0 0.00400000572323159 rpy=0 0 1.57079633736728 -> xyz=0.0022 0 0.004000006 rpy=0 0 1.570796
- joint right_finger2_joint3: origin xyz=0 0.00475028218260664 0.0436176566595782 rpy=0 0 -1.57106495008262 -> xyz=0 0.004750282 0.04361766 rpy=0 0 -1.571065
- joint right_finger2_joint4: origin xyz=0 -0.00020000000636031 0.0294999999999844 rpy=0 0 0 -> xyz=0 -0.0002 0.0295 rpy=0 0 0
- joint right_finger2_tip_fixed: axis 0 0 0 -> (none); origin xyz=-0.00104999999940632 0.000200000000000138 0.0266999989308851 rpy=0 0 0 -> xyz=-0.00105 0.0002 0.0267 rpy=0 0 0
- joint right_finger3_joint1: origin xyz=-0.0104597238611628 0.00746146014385576 0.0895435117703666 rpy=-5.08864726421373E-05 -0.0872664633653732 0.000583871740007801 -> xyz=-0.01046 0.0074615 0.089544 rpy=-5.0886e-05 -0.087266 0.00058387
- joint right_finger3_joint2: limit lower=-0.37 upper=0.37 effort=0.1827 velocity=8.1158 -> lower=-0.3700 upper=0.3700 effort=0.1827 velocity=8.115; origin xyz=0.00220000049491006 0 0.00400000560544524 rpy=0 0 1.57079633736875 -> xyz=0.0022 0 0.004000006 rpy=0 0 1.570796
- joint right_finger3_joint3: origin xyz=0 0.0047500001855858 0.0436176873657041 rpy=0 0 -1.57106495008262 -> xyz=0 0.00475 0.04361769 rpy=0 0 -1.571065
- joint right_finger3_joint4: limit lower=-0.4684 upper=1.5745 effort=0.2018 velocity=13.579 -> lower=-0.4684 upper=1.5745 effort=0.2018 velocity=13.578; origin xyz=0 -0.000200000004070615 0.0294999999999999 rpy=0 0 0 -> xyz=0 -0.0002 0.0295 rpy=0 0 0
- joint right_finger3_tip_fixed: axis 0 0 0 -> (none); origin xyz=-0.00104908716153243 0.000201039517772421 0.0266999998992792 rpy=0 0 0 -> xyz=-0.001049087 0.0002010395 0.0267 rpy=0 0 0
- joint right_finger4_joint1: origin xyz=-0.0076648599285041 -0.0137122383759844 0.084428694586379 rpy=0.0903746211775801 -0.0834355030065636 0.0471266290291302 -> xyz=-0.0076649 -0.013712 0.084429 rpy=0.090375 -0.083436 0.047127
- joint right_finger4_joint2: limit lower=-0.37 upper=0.37 effort=0.1832 velocity=8.1158 -> lower=-0.3700 upper=0.3700 effort=0.1832 velocity=8.115; origin xyz=0.00220000052979842 0 0.00400000547923511 rpy=0 0 1.57079633736852 -> xyz=0.002200001 0 0.004000005 rpy=0 0 1.570796
- joint right_finger4_joint3: origin xyz=0 0.00474999949683786 0.0436176874505065 rpy=0 0 -1.57106495008262 -> xyz=0 0.004749999 0.04361769 rpy=0 0 -1.571065
- joint right_finger4_joint4: limit lower=-0.4777 upper=1.5634 effort=0.2044 velocity=13.579 -> lower=-0.4777 upper=1.5634 effort=0.2044 velocity=13.578; origin xyz=0 -0.000200000003294468 0.0294999999999999 rpy=0 0 0 -> xyz=0 -0.0002 0.0295 rpy=0 0 0
- joint right_finger4_tip_fixed: axis 0 0 0 -> (none); origin xyz=-0.00105960974768627 0.000190450796499008 0.0266999999370233 rpy=0 0 0 -> xyz=-0.00105961 0.0001904508 0.0267 rpy=0 0 0
- joint right_finger5_joint1: origin xyz=-0.00226865106062467 -0.0340011106648613 0.0742813381426987 rpy=0.192483658660879 -0.0925172337475744 0.157672818669672 -> xyz=-0.002268651 -0.03400111 0.07428134 rpy=0.1924837 -0.09251723 0.1576728
- joint right_finger5_joint2: limit lower=-0.37 upper=0.37 effort=0.1798 velocity=8.1158 -> lower=-0.3700 upper=0.3700 effort=0.1798 velocity=8.115; origin xyz=0.0022000006995556 0 0.0040000052791524 rpy=0 0 1.5707963373693 -> xyz=0.002200001 0 0.004000005 rpy=0 0 1.570796
- joint right_finger5_joint3: origin xyz=0 0.00474999944502474 0.0436176874505066 rpy=0 0 -1.57106495008262 -> xyz=0 0.004749999 0.04361769 rpy=0 0 -1.571065
- joint right_finger5_joint4: limit lower=-0.4683 upper=1.5735 effort=0.1866 velocity=13.579 -> lower=-0.4683 upper=1.5735 effort=0.1866 velocity=13.578; origin xyz=0 -0.000200000003294461 0.0294999999999999 rpy=0 0 0 -> xyz=0 -0.0002 0.0295 rpy=0 0 0
- joint right_finger5_tip_fixed: axis 0 0 0 -> (none); origin xyz=-0.00104463936847252 0.000211309529000607 0.0267000001662517 rpy=0 0 0 -> xyz=-0.001044639 0.0002113095 0.0267 rpy=0 0 0

File: urdf/right.urdf (robot description, URDF)
Before this commit: robot wujihand-right, 26 links, 25 joints
Joints:
- joint right_finger1_joint1: origin xyz=0.0084398536891496 0.0205866432770798 0.0288928344360424 rpy=-1.32802443797267 -0.371613529401197 -0.730700470955738 -> xyz=0.0084399 0.020587 0.028893 rpy=-1.328 -0.37161 -0.7307
- joint right_finger1_joint2: origin xyz=-0.00475489769909336 -0.00581913700106552 0.0141320977693281 rpy=0.574275025049342 0.236773483165491 -1.3381949894783 -> xyz=-0.0047549 -0.0058191 0.014132 rpy=0.57428 0.23677 -1.3382
- joint right_finger1_joint3: origin xyz=-0.000266709908258896 0.000991501558320149 0.0346656189847898 rpy=0.0490494507279648 0.017311243665607 1.23305222676766 -> xyz=-0.000266705 0.0009915016 0.03466562 rpy=0.04904945 0.01731124 1.233052
- joint right_finger1_joint4: origin xyz=0 0.000200000007014398 0.0295000000021542 rpy=0 0 0 -> xyz=0 0.0002 0.0295 rpy=0 0 0
- joint right_finger1_tip_fixed: axis 0 0 0 -> (none); origin xyz=-0.00105000000124529 -0.000200000000000502 0.0272999999978436 rpy=0 0 0 -> xyz=-0.00105 -0.0002 0.0313 rpy=0 0 0
- joint right_finger2_joint1: origin xyz=-0.00587008921485247 0.0294338632809287 0.0919165306699325 rpy=-0.110709283985856 -0.0711392458057915 -0.218224846691839 -> xyz=-0.0058701 0.029434 0.091917 rpy=-0.11071 -0.071139 -0.21822
- joint right_finger2_joint2: axis 0 0.999999999978991 0 -> 0 1 0; limit lower=-0.37 upper=0.37 effort=0.1822 velocity=8.1158 -> lower=-0.3700 upper=0.3700 effort=0.1822 velocity=8.115; origin xyz=0.00220000016749383 0 0.00400000572323159 rpy=0 0 1.57079633736728 -> xyz=0.0022 0 0.004000006 rpy=0 0 1.570796
- joint right_finger2_joint3: origin xyz=0 0.00475028218260664 0.0436176566595782 rpy=0 0 -1.57106495008262 -> xyz=0 0.004750282 0.04361766 rpy=0 0 -1.571065
- joint right_finger2_joint4: origin xyz=0 -0.00020000000636031 0.0294999999999844 rpy=0 0 0 -> xyz=0 -0.0002 0.0295 rpy=0 0 0
- joint right_finger2_tip_fixed: axis 0 0 0 -> (none); origin xyz=-0.00104999999940632 0.000200000000000138 0.0266999989308851 rpy=0 0 0 -> xyz=-0.00105 0.0002 0.0267 rpy=0 0 0
- joint right_finger3_joint1: origin xyz=-0.0104597238611628 0.00746146014385576 0.0895435117703666 rpy=-5.08864726421373E-05 -0.0872664633653732 0.000583871740007801 -> xyz=-0.01046 0.0074615 0.089544 rpy=-5.0886e-05 -0.087266 0.00058387
- joint right_finger3_joint2: limit lower=-0.37 upper=0.37 effort=0.1827 velocity=8.1158 -> lower=-0.3700 upper=0.3700 effort=0.1827 velocity=8.115; origin xyz=0.00220000049491006 0 0.00400000560544524 rpy=0 0 1.57079633736875 -> xyz=0.0022 0 0.004000006 rpy=0 0 1.570796
- joint right_finger3_joint3: origin xyz=0 0.0047500001855858 0.0436176873657041 rpy=0 0 -1.57106495008262 -> xyz=0 0.00475 0.04361769 rpy=0 0 -1.571065
- joint right_finger3_joint4: limit lower=-0.4684 upper=1.5745 effort=0.2018 velocity=13.579 -> lower=-0.4684 upper=1.5745 effort=0.2018 velocity=13.578; origin xyz=0 -0.000200000004070615 0.0294999999999999 rpy=0 0 0 -> xyz=0 -0.0002 0.0295 rpy=0 0 0
- joint right_finger3_tip_fixed: axis 0 0 0 -> (none); origin xyz=-0.00104908716153243 0.000201039517772421 0.0266999998992792 rpy=0 0 0 -> xyz=-0.001049087 0.0002010395 0.0267 rpy=0 0 0
- joint right_finger4_joint1: origin xyz=-0.0076648599285041 -0.0137122383759844 0.084428694586379 rpy=0.0903746211775801 -0.0834355030065636 0.0471266290291302 -> xyz=-0.0076649 -0.013712 0.084429 rpy=0.090375 -0.083436 0.047127
- joint right_finger4_joint2: limit lower=-0.37 upper=0.37 effort=0.1832 velocity=8.1158 -> lower=-0.3700 upper=0.3700 effort=0.1832 velocity=8.115; origin xyz=0.00220000052979842 0 0.00400000547923511 rpy=0 0 1.57079633736852 -> xyz=0.002200001 0 0.004000005 rpy=0 0 1.570796
- joint right_finger4_joint3: origin xyz=0 0.00474999949683786 0.0436176874505065 rpy=0 0 -1.57106495008262 -> xyz=0 0.004749999 0.04361769 rpy=0 0 -1.571065
- joint right_finger4_joint4: limit lower=-0.4777 upper=1.5634 effort=0.2044 velocity=13.579 -> lower=-0.4777 upper=1.5634 effort=0.2044 velocity=13.578; origin xyz=0 -0.000200000003294468 0.0294999999999999 rpy=0 0 0 -> xyz=0 -0.0002 0.0295 rpy=0 0 0
- joint right_finger4_tip_fixed: axis 0 0 0 -> (none); origin xyz=-0.00105960974768627 0.000190450796499008 0.0266999999370233 rpy=0 0 0 -> xyz=-0.00105961 0.0001904508 0.0267 rpy=0 0 0
- joint right_finger5_joint1: origin xyz=-0.00226865106062467 -0.0340011106648613 0.0742813381426987 rpy=0.192483658660879 -0.0925172337475744 0.157672818669672 -> xyz=-0.002268651 -0.03400111 0.07428134 rpy=0.1924837 -0.09251723 0.1576728
- joint right_finger5_joint2: limit lower=-0.37 upper=0.37 effort=0.1798 velocity=8.1158 -> lower=-0.3700 upper=0.3700 effort=0.1798 velocity=8.115; origin xyz=0.0022000006995556 0 0.0040000052791524 rpy=0 0 1.5707963373693 -> xyz=0.002200001 0 0.004000005 rpy=0 0 1.570796
- joint right_finger5_joint3: origin xyz=0 0.00474999944502474 0.0436176874505066 rpy=0 0 -1.57106495008262 -> xyz=0 0.004749999 0.04361769 rpy=0 0 -1.571065
- joint right_finger5_joint4: limit lower=-0.4683 upper=1.5735 effort=0.1866 velocity=13.579 -> lower=-0.4683 upper=1.5735 effort=0.1866 velocity=13.578; origin xyz=0 -0.000200000003294461 0.0294999999999999 rpy=0 0 0 -> xyz=0 -0.0002 0.0295 rpy=0 0 0
- joint right_finger5_tip_fixed: axis 0 0 0 -> (none); origin xyz=-0.00104463936847252 0.000211309529000607 0.0267000001662517 rpy=0 0 0 -> xyz=-0.001044639 0.0002113095 0.0267 rpy=0 0 0
