Commit message: fix: drop rogue limit blocks, correct docking-ros path, install mjcf/usd
Apply hotfixes to the model description on top of the sysid calibration
pass in 62b85a6:

- urdf/right.urdf, urdf/right-ros.urdf: remove spurious <limit> elements
  from the five *_finger*_tip_fixed joints. URDF <limit> is only defined
  for revolute/prismatic joints; these 25 lines were the entire structural
  asymmetry between the left and right hand URDFs, which defeats the
  stated purpose of this branch. Root cause lives in the upstream
  urdf_cali pipeline (update_joint_limits.py) and is filed separately.

- docking/urdf/docking-ros.urdf: fix wrong ROS package reference. Mesh
  paths now use package://wuji_hand_description/docking/meshes/... to
  match the installed share/ layout. Previous package://wuji_description/
  robots/docking/meshes/... would have failed to resolve after colcon
  build because the package name is wuji_hand_description and there is
  no robots/ prefix.

- CMakeLists.txt: also install mjcf/ and usd/ so MuJoCo and Isaac Sim
  assets ship with the ROS package.

- README.md: document how to preview the new docking module.

- CHANGELOG.md: add entries for all of the above under [Unreleased].

Co-Authored-By: Claude Opus 4.6 (1M context) <noreply@anthropic.com>

File: docking/urdf/docking-ros.urdf (robot description, URDF)
Before this commit: robot wuji-hand-description-docking, 1 links, 0 joints
Links:
- link hand_docking_link: geometry collision mesh filename=package://wuji_hand_description/docking/meshes/hand_docking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; visual mesh filename=package://wuji_hand_description/docking/meshes/hand_docking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

File: urdf/right-ros.urdf (robot description, URDF)
Before this commit: robot wujihand-right, 26 links, 25 joints
Joints:
- joint right_finger1_tip_fixed: limit lower=0 upper=0 effort=100 velocity=10 -> (none)
- joint right_finger2_tip_fixed: limit lower=0 upper=0 effort=100 velocity=10 -> (none)
- joint right_finger3_tip_fixed: limit lower=0 upper=0 effort=100 velocity=10 -> (none)
- joint right_finger4_tip_fixed: limit lower=0 upper=0 effort=100 velocity=10 -> (none)
- joint right_finger5_tip_fixed: limit lower=0 upper=0 effort=100 velocity=10 -> (none)

File: urdf/right.urdf (robot description, URDF)
Before this commit: robot wujihand-right, 26 links, 25 joints
Joints:
- joint right_finger1_tip_fixed: limit lower=0 upper=0 effort=100 velocity=10 -> (none)
- joint right_finger2_tip_fixed: limit lower=0 upper=0 effort=100 velocity=10 -> (none)
- joint right_finger3_tip_fixed: limit lower=0 upper=0 effort=100 velocity=10 -> (none)
- joint right_finger4_tip_fixed: limit lower=0 upper=0 effort=100 velocity=10 -> (none)
- joint right_finger5_tip_fixed: limit lower=0 upper=0 effort=100 velocity=10 -> (none)
